Commit message: v2: add new modules and updates

File: Universal_Robots_ROS2_Tutorials/my_robot_cell/my_robot_cell_control/urdf/hiltest_robot_cell.urdf.xacro (robot description, xacro)
@@ -14,5 +14,5 @@
   <xacro:arg name="physical_params" default="$(find my_robot_cell_control)/config/$(arg ur_type)/physical_parameters.yaml"/>
   <xacro:arg name="visual_params" default="$(find my_robot_cell_control)/config/$(arg ur_type)/visual_parameters.yaml"/>
-  <xacro:arg name="robot_ip" default="192.168.4.5"/>
+  <xacro:arg name="robot_ip" default="192.168.3.5"/>
   <xacro:arg name="headless_mode" default="false" />
   <xacro:arg name="ur_script_filename" default="$(find ur_client_library)/resources/external_control.urscript"/>

File: Universal_Robots_ROS2_Tutorials/my_robot_cell/my_robot_cell_control/urdf/my_robot_cell_controlled.urdf.xacro (robot description, xacro)
@@ -13,5 +13,5 @@
   <xacro:arg name="physical_params" default="$(find my_robot_cell_control)/config/$(arg ur_type)/physical_parameters.yaml"/>
   <xacro:arg name="visual_params" default="$(find my_robot_cell_control)/config/$(arg ur_type)/visual_parameters.yaml"/>
-  <xacro:arg name="robot_ip" default="192.168.4.5"/>
+  <xacro:arg name="robot_ip" default="192.168.3.5"/>
   <xacro:arg name="headless_mode" default="false" />
   <xacro:arg name="ur_script_filename" default="$(find ur_client_library)/resources/external_control.urscript"/>

File: Universal_Robots_ROS2_Tutorials/my_robot_cell/my_robot_cell_description/urdf/my_robot_cell_macro.xacro (robot description, xacro)
@@ -2,4 +2,5 @@
 <robot xmlns:xacro="http://ros.org/wiki/xacro">
   <xacro:include filename="$(find ur_description)/urdf/ur_macro.xacro"/>
+  <xacro:include filename="$(find my_robot_cell_description)/urdf/chassis_macro.xacro"/>
   <xacro:macro name="my_robot_cell" params="
     parent
@@ -41,4 +42,8 @@
       </collision>
     </link>
+    <!-- Chassis assembly - tüm PART1-PART44 parçalarını içerir -->
+    <!-- <xacro:chassis_assembly tf_prefix="${tf_prefix}" parent="${parent}">
+      <origin xyz="0 0 0" rpy="0 0 0"/>
+    </xacro:chassis_assembly> -->
     <link name="${tf_prefix}chassis">
       <inertial>
@@ -170,9 +175,4 @@
       <parent link="${parent}" />
       <child link="${tf_prefix}table" />
-    </joint>
-    <joint name="${tf_prefix}base_to_chassis" type="fixed">
-      <parent link="${parent}"/>
-      <child link="${tf_prefix}chassis"/>
-      <origin xyz="0 0 0" rpy="0 0 0"/>
     </joint>
     <!-- Linear axis joint - bu joint'in tam tanımı burada olmalı -->
@@ -184,4 +184,9 @@
       <limit effort="1000" lower="0.05" upper="1.95" velocity="1.25"/>
       <dynamics damping="100.0" friction="50.0"/>
+    </joint>
+    <joint name="${tf_prefix}base_to_chassis" type="fixed">
+      <parent link="${parent}"/>
+      <child link="${tf_prefix}chassis"/>
+      <origin xyz="0 0 0" rpy="0 0 0"/>
     </joint>
     <joint name="${tf_prefix}base_to_alumuniumtable" type="fixed">

File: Universal_Robots_ROS2_Tutorials/my_robot_cell/my_robot_cell_description/urdf/simrobot_my_robot_cell_macro.xacro (robot description, xacro)
@@ -2,4 +2,5 @@
 <robot xmlns:xacro="http://ros.org/wiki/xacro">
   <xacro:include filename="$(find ur_description)/urdf/simrobot_ur_macro.xacro"/>
+  <xacro:include filename="$(find my_robot_cell_description)/urdf/chassis_macro.xacro"/>
   <xacro:macro name="simrobot_my_robot_cell" params="
     parent
@@ -36,28 +37,8 @@
       </collision>
     </link>
-    <link name="${tf_prefix}chassis">
-      <inertial>
-        <origin xyz="-1.124731 1.232845 1.108302" rpy="0 0 0"/>
-        <mass value="120.90442642947052"/>
-        <inertia ixx="129.47263" ixy="-0.023527" ixz="-0.011644"
-                iyy="73.136591" iyz="-1.726202"
-                izz="85.878511"/>
-      </inertial>
-      <visual>
-        <origin xyz="0 0 0" rpy="0 0 0"/>
-        <geometry>
-          <mesh filename="file:////home/cem/colcon_ws/src/Universal_Robots_ROS2_Description/meshes/ur10e/collision/chassis.stl" scale="0.001 0.001 0.001"/>
-        </geometry>
-        <material name="chassis_material">
-          <color rgba="0.7 0.7 0.7 1"/>
-        </material>
-      </visual>
-      <collision>
-        <origin xyz="0 0 0" rpy="0 0 0"/>
-        <geometry>
-          <mesh filename="file:////home/cem/colcon_ws/src/Universal_Robots_ROS2_Description/meshes/ur10e/collision/chassis.stl" scale="0.001 0.001 0.001"/>
-        </geometry>
-      </collision>
-    </link>
+    <!-- Chassis assembly - tüm PART1-PART44 parçalarını içerir -->
+    <xacro:chassis_assembly tf_prefix="${tf_prefix}" parent="${parent}">
+      <origin xyz="0 0 0" rpy="0 0 0"/>
+    </xacro:chassis_assembly>
     <link name="${tf_prefix}robot_mount">
       <inertial>
@@ -166,9 +147,9 @@
       <child link="${tf_prefix}table" />
     </joint>
-    <joint name="${tf_prefix}base_to_chassis" type="fixed">
+    <!-- <joint name="${tf_prefix}base_to_chassis" type="fixed">
       <parent link="${parent}"/>
       <child link="${tf_prefix}chassis"/>
       <origin xyz="0 0 0" rpy="0 0 0"/>
-    </joint>
+    </joint> -->
     <!-- Linear axis joint - bu joint'in tam tanımı burada olmalı -->
     <joint name="${tf_prefix}base_to_robot_mount" type="prismatic">

File: mobile_manipulator_description/urdf/mobile_manipulator.urdf.xacro (robot description, xacro)
@@ -1,5 +1,4 @@
 <?xml version="1.0" ?>
 <robot name="robot" xmlns:xacro="http://ros.org/wiki/xacro">
-  <link name="world"/>
   <!-- RS005L makrosu -->
   <xacro:include filename="$(find mobile_manipulator_description)/urdf/khi_rs/rs005l_macro.xacro"/>
@@ -29,9 +28,6 @@
       use_fake_hardware="$(arg use_fake_hardware)"
       generate_ros2_control_tag="true"/>
-  <joint name="world_to_ota" type="fixed">
-    <parent link="world"/>
-    <child link="ota_base_link"/>
-    <origin xyz="-2.301949 0.530401 0.0" rpy="0 0 1.570796"/>
-  </joint>
+  <!-- AGV'nin hareket edebilmesi için world bağlantısı KALDIRILDI -->
+  <!-- Eğer sabit başlangıç pozisyonu istiyorsanız, spawn sırasında -x -y -z parametreleri kullanın -->
   <!-- instantiate ota -->
   <!-- <xacro:ota_base link_name="ota_base_link"/>
@@ -54,4 +50,5 @@
   </xacro:khi_rs005l>
   <xacro:if value="$(arg sim_ignition)">
+    <!-- Kawasaki robot arm controller -->
     <gazebo>
       <plugin filename="gz_ros2_control-system" name="gz_ros2_control::GazeboSimROS2ControlPlugin">
@@ -63,4 +60,11 @@
       </plugin>
     </gazebo>
+    <!-- OTA AGV diff drive controller (ayrı plugin) -->
+    <gazebo>
+      <plugin filename="gz_ros2_control-system" name="gz_ros2_control::GazeboSimROS2ControlPlugin">
+        <parameters>$(find mobile_manipulator_description)/config/ota_controllers.yaml</parameters>
+        <controller_manager_node_name>ota_controller_manager</controller_manager_node_name>
+      </plugin>
+    </gazebo>
   </xacro:if>
 </robot>

File: mobile_manipulator_description/urdf/ota/ota_macro.xacro (robot description, xacro)
@@ -82,7 +82,11 @@
         <mass value="50.0"/>
         <origin xyz="0 0 0"/>
-        <inertia ixx="1" iyy="1" izz="1" ixy="0" ixz="0" iyz="0"/>
+        <inertia ixx="5.0" iyy="5.0" izz="5.0" ixy="0" ixz="0" iyz="0"/>
       </inertial>
     </link>
+    <gazebo reference="${link_name}">
+      <mu1>0.1</mu1>
+      <mu2>0.1</mu2>
+    </gazebo>
     <link name='manipulator_base_link'>
       <origin xyz="0 0 0" rpy=" 0 0 0"/>
@@ -123,7 +127,8 @@
       <!-- === WHEEL COLLISION (simple cylinder) === -->
       <collision>
-        <origin xyz="0 0 0" rpy="0 0 0"/>
-        <geometry>
-          <cylinder radius="0.102" length="0.02"/>
+        <origin xyz="0 0 0" rpy="0 0 1.570796"/>
+        <geometry>
+          <mesh filename="file:////home/cem/colcon_ws/src/mobile_manipulator_description/meshes/ota/AnaTeker.stl"
+                scale="0.001 0.001 0.001"/>
         </geometry>
       </collision>
@@ -138,4 +143,13 @@
       <axis xyz="0 1 0"/>
     </joint>
+    <!-- Gazebo wheel parameters -->
+    <gazebo reference="wheel_${side}_link">
+      <mu1>1.0</mu1>
+      <mu2>1.0</mu2>
+      <kp>1000000.0</kp>
+      <kd>10.0</kd>
+      <minDepth>0.001</minDepth>
+      <material>Gazebo/Red</material>
+    </gazebo>
   </xacro:macro>
   <!-- OTA caster wheels -->
@@ -153,17 +167,18 @@
         <origin xyz="0 0 0"/>
         <geometry>
-          <cylinder radius="0.04" length="0.02"/>
+          <mesh filename="file:////home/cem/colcon_ws/src/mobile_manipulator_description/meshes/ota/SarhosTeker.stl"
+                scale="0.001 0.0008 0.001"/>
         </geometry>
       </collision>
       <xacro:cylinder_inertial radius="0.04" length="0.02" mass="0.5" />
     </link>
-    <!-- Bu joint continous'tu -->
+    <!-- Bu joint continous'tu ben değiştirdim-->
     <joint name="caster_${side}_joint" type="fixed">
-      <axis xyz="0 0 1"/>
+      <axis xyz="1 0 0"/>
       <origin xyz="${xyz_caster}" rpy="${rpy_caster}"/>
       <child link="caster_${side}_link"/>
       <parent link="${base_link}"/>
     </joint>
-    <link name='caster_wheel_${side}_link'>
+    <!-- <link name='caster_wheel_${side}_link'>
       <visual>
         <origin xyz="0 0 0"/>
@@ -185,5 +200,5 @@
       <parent link="caster_${side}_link"/>
       <child link="caster_wheel_${side}_link"/>
-    </joint>
+    </joint>   -->
   </xacro:macro>
   <!-- OTA IR sensor -->
@@ -250,11 +265,11 @@
     <xacro:ota_ir base_link="${base_link}" link_name="ota_ir" xyz_ir="0.503 0.0 0.175" rpy_ir="0 0 0"/>
     <!-- Tahrik tekerlekleri -->
-    <xacro:ota_wheel base_link="${base_link}" xyz_hub="0 -0.30 0.10" rpy_hub="0 0 0" side="left"/>
-    <xacro:ota_wheel base_link="${base_link}" xyz_hub="0 0.30 0.10" rpy_hub="0 0 0" side="right"/>
+    <xacro:ota_wheel base_link="${base_link}" xyz_hub="0 -0.305 0.10" rpy_hub="0 0 0" side="left"/>
+    <xacro:ota_wheel base_link="${base_link}" xyz_hub="0 0.295 0.10" rpy_hub="0 0 0" side="right"/>
     <!-- Sarhoş tekerlekler -->
-    <xacro:ota_swivel base_link="${base_link}" xyz_caster="0.37 -0.22 0.12" rpy_caster="0 0 0" side="front_right"/>
-    <xacro:ota_swivel base_link="${base_link}" xyz_caster="0.37 0.22 0.12" rpy_caster="0 0 0" side="front_left"/>
-    <xacro:ota_swivel base_link="${base_link}" xyz_caster="-0.37 -0.22 0.12" rpy_caster="0 0 0" side="back_right"/>
-    <xacro:ota_swivel base_link="${base_link}" xyz_caster="-0.37 0.22 0.12" rpy_caster="0 0 0" side="back_left"/>
+    <xacro:ota_swivel base_link="${base_link}" xyz_caster="0.37 -0.223 0.12" rpy_caster="0 0 0" side="front_right"/>
+    <xacro:ota_swivel base_link="${base_link}" xyz_caster="0.37 0.217 0.12" rpy_caster="0 0 0" side="front_left"/>
+    <xacro:ota_swivel base_link="${base_link}" xyz_caster="-0.37 -0.223 0.12" rpy_caster="0 0 0" side="back_right"/>
+    <xacro:ota_swivel base_link="${base_link}" xyz_caster="-0.37 0.217 0.12" rpy_caster="0 0 0" side="back_left"/>
   </xacro:macro>
 </robot>
