Commit message: Gripper+Conveyor

File: Universal_Robots_ROS2_Tutorials/my_robot_cell/my_robot_cell_control/urdf/my_robot_cell_controlled.urdf.xacro (robot description, xacro)
@@ -5,5 +5,5 @@
   <!--The ur_description package already provides a control tag for the UR arm, we can directly include-->
   <xacro:include filename="$(find ur_description)/urdf/ur.ros2_control.xacro"/>
-  <!-- ifarlab ortam makrosu -->
+  <!-- cem ortam makrosu -->
   <xacro:include filename="$(find mobile_manipulator_description)/urdf/ifarlab_environment.xacro"/>
   <!--We need to specify the arguments used for parametrizing our description-->
@@ -26,5 +26,5 @@
   <xacro:property name="kinematics_hash" value="${xacro.load_yaml(kinematics_params_file)['kinematics']['hash']}"/>
   <link name="world" />
-  <!-- ifarlab ortam bileşenlerini spawn et (world frame'e sabitli) -->
+  <!-- cem ortam bileşenlerini spawn et (world frame'e sabitli) -->
   <xacro:ifarlab_environment prefix=""/>
   <!--Create the scene description including the robot-->

File: Universal_Robots_ROS2_Tutorials/my_robot_cell/my_robot_cell_description/urdf/simrobot_my_robot_cell.urdf.xacro (robot description, xacro)
@@ -2,5 +2,5 @@
 <robot name="my_robot_cell_sim" xmlns:xacro="http://ros.org/wiki/xacro">
   <xacro:include filename="$(find my_robot_cell_description)/urdf/simrobot_my_robot_cell_macro.xacro"/>
-  <!-- ifarlab ortam makrosu -->
+  <!-- cem ortam makrosu -->
   <xacro:include filename="$(find mobile_manipulator_description)/urdf/ifarlab_environment.xacro"/>
   <xacro:arg name="ur_type" default="ur10e"/>
@@ -12,6 +12,7 @@
   <xacro:arg name="simulation_controllers" default="" />
   <xacro:arg name="tf_prefix" default="sim_" /> <!--sim_ur10e_ for digital twin-->
+  <xacro:arg name="use_gripper" default="false" />
   <link name="world"/>
-  <!-- ifarlab ortam bileşenlerini spawn et (world frame'e sabitli) -->
+  <!-- cem ortam bileşenlerini spawn et (world frame'e sabitli) -->
   <xacro:ifarlab_environment prefix=""/>
   <!--This will create the scene where the robot is located in-->
@@ -25,4 +26,5 @@
     sim_ignition="$(arg sim_ignition)"
     tf_prefix="$(arg tf_prefix)ur10e_"
+    use_gripper="$(arg use_gripper)"
     >
       <origin xyz="0.0 0 0" rpy="0 0 0" />

File: Universal_Robots_ROS2_Tutorials/my_robot_cell/my_robot_cell_description/urdf/simrobot_my_robot_cell_macro.xacro (robot description, xacro)
@@ -13,4 +13,5 @@
     sim_ignition:=true
     tf_prefix:='sim_ur10e_'
+    use_gripper:=false
     ">
     <material name="silver">
@@ -177,5 +178,5 @@
       </collision>
     </link>
-    <link name="${tf_prefix}conveyor_belt">
+    <!-- <link name="${tf_prefix}conveyor_belt">
       <inertial>
         <origin rpy="0 0 0" xyz="0.731215 0.101822 0.642664"/>
@@ -196,5 +197,5 @@
         </geometry>
       </collision>
-    </link>
+    </link> -->
     <!-- Joint tanımları -->
     <joint name="${tf_prefix}table_base_joint" type="fixed">
@@ -239,9 +240,9 @@
       <origin xyz="0 0 0" rpy="0 0 0"/>
     </joint>
-    <joint name="${tf_prefix}base_to_conveyorbelt" type="fixed">
+    <!-- <joint name="${tf_prefix}base_to_conveyorbelt" type="fixed">
       <parent link="${parent}"/>
       <child link="${tf_prefix}conveyor_belt"/>
       <origin xyz="0 0 0" rpy="0 0 0"/>
-    </joint>
+    </joint> -->
     <link name="${tf_prefix}stackable_bin">
       <inertial>
@@ -328,4 +329,5 @@
       generate_ros2_control_tag="true"
       sim_ignition="${sim_ignition}"
+      use_gripper="${use_gripper}"
     >
       <origin xyz="0 0 0" rpy="0 0 0" />

File: mobile_manipulator_description/urdf/ota/ota_base.xacro (robot description, xacro)
@@ -85,5 +85,5 @@
       </visual>
     </gazebo> -->
-    <!-- ifarlab.sdf: ifarlab_ray model pose = "0 0 0 0 0 0" → world origin -->
+    <!-- cem.sdf: ifarlab_ray model pose = "0 0 0 0 0 0" → world origin -->
     <joint name="ifarlab_ray_joint" type="fixed">
       <parent link="world"/>
@@ -91,5 +91,5 @@
       <origin xyz="0 0 0" rpy="0 0 0"/>
     </joint>
-    <!-- AGV başlangıç konumu: ifarlab.sdf spawn pozisyonundan okundu
+    <!-- AGV başlangıç konumu: cem.sdf spawn pozisyonundan okundu
          x=-2.301949  y=0.135135131  z=0.17  yaw=1.570796 (90°)
          axis 1 0 0 = joint frame local X = yaw 90° nedeniyle world +Y yönü
