Commit message: Dual 7 axis robot systems

File: Universal_Robots_ROS2_Tutorials/my_robot_cell/my_robot_cell_control/urdf/whole_cell_sim.urdf.xacro (robot description, xacro)
@@ -56,5 +56,5 @@
   <!-- Kawasaki argümanları -->
   <xacro:arg name="kawasaki_name" default="rs005l"/>
-  <xacro:arg name="kawasaki_tf_prefix" default=""/>
+  <xacro:arg name="kawasaki_tf_prefix" default="sim_kawasaki_"/>
   <xacro:arg name="kawasaki_sim_ignition" default="true"/>
   <xacro:arg name="kawasaki_use_fake_hardware" default="false"/>

File: rs005l_description/urdf/rs005l.ros2_control.xacro (robot description, xacro)
@@ -22,30 +22,30 @@
       </hardware>
       <!-- orjinalinde command interface effort bunu sormak lazım -->
-      <joint name="joint1">
+      <joint name="${tf_prefix}joint1">
         <command_interface name="position"/>
         <state_interface name="position"/>
         <state_interface name="velocity"/>
       </joint>
-      <joint name="joint2">
+      <joint name="${tf_prefix}joint2">
         <command_interface name="position"/>
         <state_interface name="position"/>
         <state_interface name="velocity"/>
       </joint>
-      <joint name="joint3">
+      <joint name="${tf_prefix}joint3">
         <command_interface name="position"/>
         <state_interface name="position"/>
         <state_interface name="velocity"/>
       </joint>
-      <joint name="joint4">
+      <joint name="${tf_prefix}joint4">
         <command_interface name="position"/>
         <state_interface name="position"/>
         <state_interface name="velocity"/>
       </joint>
-      <joint name="joint5">
+      <joint name="${tf_prefix}joint5">
         <command_interface name="position"/>
         <state_interface name="position"/>
         <state_interface name="velocity"/>
       </joint>
-      <joint name="joint6">
+      <joint name="${tf_prefix}joint6">
         <command_interface name="position"/>
         <state_interface name="position"/>
