Commit message: Kawasaki ros2_control

File: Universal_Robots_ROS2_Tutorials/my_robot_cell/my_robot_cell_control/urdf/whole_cell_sim.urdf.xacro (robot description, xacro)
@@ -76,22 +76,23 @@
   </joint> -->
   <!-- AGV gövdesi -->
-  <xacro:ota_base link_name="ota_base_link"/>
+  <xacro:ota_base link_name="sim_ota_base_link" prefix="sim_"/>
   <!-- AGV ros2_control (tekerlek velocity interface) -->
   <xacro:ota_ros2_control
     name="ota_system"
     sim_ignition="$(arg kawasaki_sim_ignition)"
-    use_fake_hardware="$(arg kawasaki_use_fake_hardware)"/>
+    use_fake_hardware="$(arg kawasaki_use_fake_hardware)"
+    prefix="sim_"/>
   <!-- IR sensör -->
-  <xacro:ota_ir base_link="ota_base_link" link_name="ota_ir" xyz_ir="0.403 0.0 0.03" rpy_ir="0 0 0"/>
+  <xacro:ota_ir base_link="sim_ota_base_link" link_name="sim_ota_ir" xyz_ir="0.403 0.0 0.03" rpy_ir="0 0 0"/>
   <!-- Tahrik tekerlekleri -->
-  <xacro:ota_wheel base_link="ota_base_link" xyz_hub="0 -0.30 -0.06" rpy_hub="0 0 0" side="left"/>
-  <xacro:ota_wheel base_link="ota_base_link" xyz_hub="0 0.30 -0.06" rpy_hub="0 0 0" side="right"/>
+  <xacro:ota_wheel base_link="sim_ota_base_link" xyz_hub="0 -0.30 -0.06" rpy_hub="0 0 0" side="left" prefix="sim_"/>
+  <xacro:ota_wheel base_link="sim_ota_base_link" xyz_hub="0 0.30 -0.06" rpy_hub="0 0 0" side="right" prefix="sim_"/>
   <!-- Sarhoş tekerlekler -->
-  <xacro:ota_swivel base_link="ota_base_link" xyz_caster="0.37 -0.22 -0.048" rpy_caster="0 0 0" side="front_right"/>
-  <xacro:ota_swivel base_link="ota_base_link" xyz_caster="0.37 0.22 -0.048" rpy_caster="0 0 0" side="front_left"/>
-  <xacro:ota_swivel base_link="ota_base_link" xyz_caster="-0.37 -0.22 -0.048" rpy_caster="0 0 0" side="back_right"/>
-  <xacro:ota_swivel base_link="ota_base_link" xyz_caster="-0.37 0.22 -0.048" rpy_caster="0 0 0" side="back_left"/>
+  <xacro:ota_swivel base_link="sim_ota_base_link" xyz_caster="0.37 -0.22 -0.048" rpy_caster="0 0 0" side="front_right" prefix="sim_"/>
+  <xacro:ota_swivel base_link="sim_ota_base_link" xyz_caster="0.37 0.22 -0.048" rpy_caster="0 0 0" side="front_left" prefix="sim_"/>
+  <xacro:ota_swivel base_link="sim_ota_base_link" xyz_caster="-0.37 -0.22 -0.048" rpy_caster="0 0 0" side="back_right" prefix="sim_"/>
+  <xacro:ota_swivel base_link="sim_ota_base_link" xyz_caster="-0.37 0.22 -0.048" rpy_caster="0 0 0" side="back_left" prefix="sim_"/>
   <!-- Diff Drive Plugin (AGV hareketi için) -->
-  <xacro:ota_diff_drive base_link="ota_base_link"/>
+  <xacro:ota_diff_drive base_link="sim_ota_base_link" prefix="sim_"/>
   <!-- Joint State Publisher Plugin -->
   <xacro:ota_joints_state_publisher/>
@@ -100,5 +101,5 @@
     name="$(arg kawasaki_name)"
     tf_prefix="$(arg kawasaki_tf_prefix)"
-    parent="manipulator_base_link"
+    parent="sim_manipulator_base_link"
     sim_ignition="$(arg kawasaki_sim_ignition)"
     use_fake_hardware="$(arg kawasaki_use_fake_hardware)">

File: Universal_Robots_ROS2_Tutorials/my_robot_cell/my_robot_cell_description/urdf/my_robot_cell_macro.xacro (robot description, xacro)
@@ -203,7 +203,7 @@
     <link name="${tf_prefix}alumunium_table">
       <inertial>
-        <origin rpy="0 0 0" xyz="681.141 2464.643 737.851"/>
-        <mass value="20.04925448455695"/>
-        <inertia ixx="130.9" ixy="0.04503" ixz="0.9303" iyy="70.758" iyz="-0.03313" izz="139.1"/>
+        <origin rpy="0 0 0" xyz="0.713931 2.546776 0.955293"/>
+        <mass value="82.723802"/>
+        <inertia ixx="21.46" ixy="-0.6779" ixz="-0.1229" iyy="14.70" iyz="-2.239" izz="16.12"/>
       </inertial>
       <visual>
@@ -221,9 +221,49 @@
       </collision>
     </link>
+    <link name="${tf_prefix}screwdriver">
+      <inertial>
+        <origin rpy="0 0 0" xyz="0.698999 2.916019 1.646605"/>
+        <mass value="2.400984"/>
+        <inertia ixx="0.004047" ixy="-4.087e-08" ixz="-1.236e-07" iyy="0.004295" iyz="2.148e-05" izz="0.001060"/>
+      </inertial>
+      <visual>
+        <origin rpy="0 0 0" xyz="0 0 0"/>
+        <geometry>
+          <mesh filename="file:////home/cem/colcon_ws/src/Universal_Robots_ROS2_Description/meshes/ur10e/collision/screwdriver.stl" scale="0.001 0.001 0.001"/>
+        </geometry>
+        <material name="silver"/>
+      </visual>
+      <collision>
+        <origin rpy="0 0 0" xyz="0 0 0"/>
+        <geometry>
+          <mesh filename="file:////home/cem/colcon_ws/src/Universal_Robots_ROS2_Description/meshes/ur10e/collision/screwdriver.stl" scale="0.001 0.001 0.001"/>
+        </geometry>
+      </collision>
+    </link>
+    <link name="${tf_prefix}screw_feeder">
+      <inertial>
+        <origin rpy="0 0 0" xyz="0.47973 2.996281 0.677038"/>
+        <mass value="64.903172"/>
+        <inertia ixx="5.385" ixy="3.3487e-05" ixz="-0.03657" iyy="5.631" iyz="0.003393" izz="0.4777"/>
+      </inertial>
+      <visual>
+        <origin rpy="0 0 0" xyz="0 0 0"/>
+        <geometry>
+          <mesh filename="file:////home/cem/colcon_ws/src/Universal_Robots_ROS2_Description/meshes/ur10e/collision/screw_feeder.stl" scale="0.001 0.001 0.001"/>
+        </geometry>
+        <material name="silver"/>
+      </visual>
+      <collision>
+        <origin rpy="0 0 0" xyz="0 0 0"/>
+        <geometry>
+          <mesh filename="file:////home/cem/colcon_ws/src/Universal_Robots_ROS2_Description/meshes/ur10e/collision/screw_feeder.stl" scale="0.001 0.001 0.001"/>
+        </geometry>
+      </collision>
+    </link>
     <link name="${tf_prefix}conveyor_belt">
       <inertial>
-        <origin rpy="0 0 0" xyz="736.828 104.977 664.295"/>
-        <mass value="15.04925448455695"/>
-        <inertia ixx="0.061984" ixy="-0.003503" ixz="0.001551" iyy="0.069314" iyz="0.000564" izz="0.125682"/>
+        <origin rpy="0 0 0" xyz="0.651237 0.086681 0.615798"/>
+        <mass value="26.689341"/>
+        <inertia ixx="3.942" ixy="-0.008312" ixz="-0.009881" iyy="2.162" iyz="0.06187" izz="2.363"/>
       </inertial>
       <visual>
@@ -307,4 +347,14 @@
       <parent link="${parent}"/>
       <child link="${tf_prefix}alumunium_table"/>
+      <origin xyz="0 0 0" rpy="0 0 0"/>
+    </joint>
+    <joint name="${tf_prefix}base_to_screwdriver" type="fixed">
+      <parent link="${parent}"/>
+      <child link="${tf_prefix}screwdriver"/>
+      <origin xyz="0 0 0" rpy="0 0 0"/>
+    </joint>
+    <joint name="${tf_prefix}base_to_screw_feeder" type="fixed">
+      <parent link="${parent}"/>
+      <child link="${tf_prefix}screw_feeder"/>
       <origin xyz="0 0 0" rpy="0 0 0"/>
     </joint>

File: Universal_Robots_ROS2_Tutorials/my_robot_cell/my_robot_cell_description/urdf/simrobot_my_robot_cell_macro.xacro (robot description, xacro)
@@ -160,7 +160,7 @@
     <link name="${tf_prefix}alumunium_table">
       <inertial>
-        <origin rpy="0 0 0" xyz="0.681141 2.464643 0.737851"/>
-        <mass value="20.04925448455695"/>
-        <inertia ixx="130.9" ixy="0.04503" ixz="0.9303" iyy="70.758" iyz="-0.03313" izz="139.1"/>
+        <origin rpy="0 0 0" xyz="0.713931 2.546776 0.955293"/>
+        <mass value="82.723802"/>
+        <inertia ixx="21.46" ixy="-0.6779" ixz="-0.1229" iyy="14.70" iyz="-2.239" izz="16.12"/>
       </inertial>
       <visual>
@@ -178,9 +178,49 @@
       </collision>
     </link>
+    <link name="${tf_prefix}screwdriver">
+      <inertial>
+        <origin rpy="0 0 0" xyz="0.698999 2.916019 1.646605"/>
+        <mass value="2.400984"/>
+        <inertia ixx="0.004047" ixy="-4.087e-08" ixz="-1.236e-07" iyy="0.004295" iyz="2.148e-05" izz="0.001060"/>
+      </inertial>
+      <visual>
+        <origin rpy="0 0 0" xyz="0 0 0"/>
+        <geometry>
+          <mesh filename="file:////home/cem/colcon_ws/src/Universal_Robots_ROS2_Description/meshes/ur10e/collision/screwdriver.stl" scale="0.001 0.001 0.001"/>
+        </geometry>
+        <material name="silver"/>
+      </visual>
+      <collision>
+        <origin rpy="0 0 0" xyz="0 0 0"/>
+        <geometry>
+          <mesh filename="file:////home/cem/colcon_ws/src/Universal_Robots_ROS2_Description/meshes/ur10e/collision/screwdriver.stl" scale="0.001 0.001 0.001"/>
+        </geometry>
+      </collision>
+    </link>
+    <link name="${tf_prefix}screw_feeder">
+      <inertial>
+        <origin rpy="0 0 0" xyz="0.47973 2.996281 0.677038"/>
+        <mass value="64.903172"/>
+        <inertia ixx="5.385" ixy="3.3487e-05" ixz="-0.03657" iyy="5.631" iyz="0.003393" izz="0.4777"/>
+      </inertial>
+      <visual>
+        <origin rpy="0 0 0" xyz="0 0 0"/>
+        <geometry>
+          <mesh filename="file:////home/cem/colcon_ws/src/Universal_Robots_ROS2_Description/meshes/ur10e/collision/screw_feeder.stl" scale="0.001 0.001 0.001"/>
+        </geometry>
+        <material name="silver"/>
+      </visual>
+      <collision>
+        <origin rpy="0 0 0" xyz="0 0 0"/>
+        <geometry>
+          <mesh filename="file:////home/cem/colcon_ws/src/Universal_Robots_ROS2_Description/meshes/ur10e/collision/screw_feeder.stl" scale="0.001 0.001 0.001"/>
+        </geometry>
+      </collision>
+    </link>
     <!-- <link name="${tf_prefix}conveyor_belt">
       <inertial>
-        <origin rpy="0 0 0" xyz="0.731215 0.101822 0.642664"/>
-        <mass value="27.036586"/>
-        <inertia ixx="4.104" ixy="-0.008305" ixz="-0.010260" iyy="2.304" iyz="0.064250" izz="2.392"/>
+        <origin rpy="0 0 0" xyz="0.651237 0.086681 0.615798"/>
+        <mass value="26.689341"/>
+        <inertia ixx="3.942" ixy="-0.008312" ixz="-0.009881" iyy="2.162" iyz="0.06187" izz="2.363"/>
       </inertial>
       <visual>
@@ -238,4 +278,14 @@
       <parent link="${parent}"/>
       <child link="${tf_prefix}alumunium_table"/>
+      <origin xyz="0 0 0" rpy="0 0 0"/>
+    </joint>
+    <joint name="${tf_prefix}base_to_screwdriver" type="fixed">
+      <parent link="${parent}"/>
+      <child link="${tf_prefix}screwdriver"/>
+      <origin xyz="0 0 0" rpy="0 0 0"/>
+    </joint>
+    <joint name="${tf_prefix}base_to_screw_feeder" type="fixed">
+      <parent link="${parent}"/>
+      <child link="${tf_prefix}screw_feeder"/>
       <origin xyz="0 0 0" rpy="0 0 0"/>
     </joint>

File: mobile_manipulator_description/urdf/ota/ota.ros2_control.xacro (robot description, xacro)
@@ -7,4 +7,5 @@
       generate_ros2_control_tag:=true
       fake_sensor_commands:=false
+      prefix:=''
     ">
     <xacro:if value="${generate_ros2_control_tag}">
@@ -19,7 +20,13 @@
             <param name="state_following_offset">0.0</param>
           </xacro:if>
+          <xacro:if value="${not sim_ignition and not use_fake_hardware}">
+            <plugin>topic_based_ros2_control/TopicBasedSystem</plugin>
+            <param name="joint_commands_topic">/agv/joint_cmd</param>
+            <param name="joint_states_topic">/joint_states</param>
+            <param name="sum_wrapped_joint_states">true</param>
+          </xacro:if>
         </hardware>
         <!-- Right wheel -->
-        <joint name="wheel_right_base">
+        <joint name="${prefix}wheel_right_base">
           <command_interface name="velocity"/>
           <state_interface name="position"/>
@@ -27,21 +34,26 @@
         </joint>
         <!-- Left wheel -->
-        <joint name="wheel_left_base">
+        <joint name="${prefix}wheel_left_base">
           <command_interface name="velocity"/>
           <state_interface name="position"/>
           <state_interface name="velocity"/>
         </joint>
-        <joint name="world_to_agv">
-          <command_interface name="position"/>
-          <command_interface name="velocity">
-            <param name="min">-1.25</param>
-            <param name="max">1.25</param>
-          </command_interface>
-          <state_interface name="position">
-              <param name="initial_value">1.0</param>
-          </state_interface>
-          <state_interface name="velocity"/>
-          <state_interface name="effort"/>
-        </joint>
+        <!-- world_to_agv:
+             - fake hardware → rs005l GenericSystem altında (7-DOF tek system)
+             - gerçek hardware → ota_system TopicBasedSystem altında -->
+        <xacro:unless value="${use_fake_hardware}">
+          <joint name="${prefix}world_to_agv">
+            <command_interface name="position"/>
+            <command_interface name="velocity">
+              <param name="min">-1.25</param>
+              <param name="max">1.25</param>
+            </command_interface>
+            <state_interface name="position">
+                <param name="initial_value">1.0</param>
+            </state_interface>
+            <state_interface name="velocity"/>
+            <state_interface name="effort"/>
+          </joint>
+        </xacro:unless>
       </ros2_control>
     </xacro:if>

File: mobile_manipulator_description/urdf/ota/ota_base.xacro (robot description, xacro)
@@ -1,7 +1,7 @@
 <?xml version='1.0'?>
 <robot xmlns:xacro="http://ros.org/wiki/xacro">
-  <xacro:macro name="ota_base" params="link_name">
+  <xacro:macro name="ota_base" params="link_name prefix:=''">
     <!-- <link name="world"/> -->
-    <link name="ifarlab_ray_link">
+    <link name="${prefix}ifarlab_ray_link">
       <inertial>
         <mass value="1.0"/>
@@ -12,5 +12,5 @@
           <mesh filename="file://$(find mobile_manipulator_description)/meshes/environment/ifarlab_ray.stl" scale="0.001 0.001 0.001"/>
         </geometry>
-        <material name="ifarlab_ray_material">
+        <material name="${prefix}ifarlab_ray_material">
           <color rgba="0.75 0.75 0.75 1"/>
         </material>
@@ -29,5 +29,5 @@
           <mesh filename="file:////home/cem/colcon_ws/src/mobile_manipulator_description/meshes/ota/OTA-v0.7.stl" scale="0.001 0.001 0.001"/>
         </geometry>
-        <material name="DefaultWhite">
+        <material name="${prefix}DefaultWhite">
           <color rgba="1 1 1 1"/>
         </material>
@@ -59,5 +59,5 @@
       </visual>
     </gazebo>
-    <link name='manipulator_base_link'>
+    <link name='${prefix}manipulator_base_link'>
       <origin xyz="0 0 0" rpy=" 0 0 0"/>
       <visual>
@@ -75,5 +75,5 @@
       <xacro:box_inertial x="0.187945" y="0.190701"  z="0.103" mass="5.0" />
     </link>
-    <!-- <gazebo reference="manipulator_base_link">
+    <!-- <gazebo reference="${prefix}manipulator_base_link">
       <material>Gazebo/Orange</material>
       <visual>
@@ -86,7 +86,7 @@
     </gazebo> -->
     <!-- cem.sdf: ifarlab_ray model pose = "0 0 0 0 0 0" → world origin -->
-    <joint name="ifarlab_ray_joint" type="fixed">
+    <joint name="${prefix}ifarlab_ray_joint" type="fixed">
       <parent link="world"/>
-      <child link="ifarlab_ray_link"/>
+      <child link="${prefix}ifarlab_ray_link"/>
       <origin xyz="0 0 0" rpy="0 0 0"/>
     </joint>
@@ -95,6 +95,6 @@
          axis 1 0 0 = joint frame local X = yaw 90° nedeniyle world +Y yönü
          Bu eksende AGV ileri/geri hareket eder (ray üzerinde kayar) -->
-    <joint name="world_to_agv" type="prismatic">
-      <parent link="ifarlab_ray_link"/>
+    <joint name="${prefix}world_to_agv" type="prismatic">
+      <parent link="${prefix}ifarlab_ray_link"/>
       <child link="${link_name}"/>
       <origin xyz="-2.301959 0.135135131 0.165" rpy="0 0 1.570796"/>
@@ -103,7 +103,7 @@
       <dynamics damping="100.0" friction="50.0"/>
     </joint>
-    <joint name="base2manipulatorbase" type="fixed">
+    <joint name="${prefix}base2manipulatorbase" type="fixed">
       <parent link="${link_name}"/>
-      <child link="manipulator_base_link"/>
+      <child link="${prefix}manipulator_base_link"/>
       <origin rpy="0 0 0" xyz="0.001 -0.26 0.212"/>
     </joint>

File: mobile_manipulator_description/urdf/ota/ota_caster.xacro (robot description, xacro)
@@ -2,7 +2,7 @@
 <robot xmlns:xacro="http://www.ros.org/wiki/xacro">
   <property name="M_PI" value="3.1415926535897931" />
-  <xacro:macro name="ota_swivel" params="base_link xyz_caster rpy_caster side">
+  <xacro:macro name="ota_swivel" params="base_link xyz_caster rpy_caster side prefix:=''">
     <!-- CASTER BODY -->
-    <link name='caster_${side}_link'>
+    <link name='${prefix}caster_${side}_link'>
       <visual>
         <origin xyz="0 0 0"/>
@@ -27,11 +27,11 @@
       </inertial>
     </link>
-    <joint name="caster_${side}_joint" type="fixed">
+    <joint name="${prefix}caster_${side}_joint" type="fixed">
       <axis xyz="0 0 1"/>
       <origin xyz="${xyz_caster}" rpy="${rpy_caster}"/>
-      <child link="caster_${side}_link"/>
+      <child link="${prefix}caster_${side}_link"/>
       <parent link="${base_link}"/>
     </joint>
-    <gazebo reference="caster_${side}_link">
+    <gazebo reference="${prefix}caster_${side}_link">
       <mu1>1.0</mu1>
       <mu2>1.0</mu2>
@@ -48,5 +48,5 @@
       </visual>
     </gazebo>
-    <link name='caster_wheel_${side}_link'>
+    <link name='${prefix}caster_wheel_${side}_link'>
       <visual>
         <origin xyz="0 0 0"/>
@@ -70,9 +70,9 @@
       </inertial>
     </link>
-    <joint name="caster_${side}_wheel_joint" type="fixed">
+    <joint name="${prefix}caster_${side}_wheel_joint" type="fixed">
       <axis xyz="0 1 0"/>
       <origin xyz="-0.04 0 -0.07"/>
-      <parent link="caster_${side}_link"/>
-      <child link="caster_wheel_${side}_link"/>
+      <parent link="${prefix}caster_${side}_link"/>
+      <child link="${prefix}caster_wheel_${side}_link"/>
     </joint>
   </xacro:macro>

File: mobile_manipulator_description/urdf/ota/ota_macro.xacro (robot description, xacro)
@@ -13,4 +13,5 @@
     sim_ignition:=false
     generate_ros2_control_tag:=true
+    prefix:=''
     ">
     <xacro:if value="${generate_ros2_control_tag}">
@@ -22,18 +23,19 @@
         use_fake_hardware="${use_fake_hardware}"
         sim_ignition="${sim_ignition}"
+        prefix="${prefix}"
       />
     </xacro:if>
     <!-- AGV gövdesi -->
-    <xacro:ota_base link_name="${base_link}"/>
+    <xacro:ota_base link_name="${base_link}" prefix="${prefix}"/>
     <!-- IR sensör -->
-    <xacro:ota_ir base_link="${base_link}" link_name="ota_ir" xyz_ir="0.403 0.0 0.03" rpy_ir="0 0 0"/>
+    <xacro:ota_ir base_link="${base_link}" link_name="${prefix}ota_ir" xyz_ir="0.403 0.0 0.03" rpy_ir="0 0 0"/>
     <!-- Tahrik tekerlekleri -->
-    <xacro:ota_wheel base_link="${base_link}" xyz_hub="0 -0.30 -0.06" rpy_hub="0 0 0" side="left"/>
-    <xacro:ota_wheel base_link="${base_link}" xyz_hub="0 0.30 -0.06" rpy_hub="0 0 0" side="right"/>
+    <xacro:ota_wheel base_link="${base_link}" xyz_hub="0 -0.30 -0.06" rpy_hub="0 0 0" side="left" prefix="${prefix}"/>
+    <xacro:ota_wheel base_link="${base_link}" xyz_hub="0 0.30 -0.06" rpy_hub="0 0 0" side="right" prefix="${prefix}"/>
     <!-- Sarhoş tekerlekler -->
-    <xacro:ota_swivel base_link="${base_link}" xyz_caster="0.37 -0.22 -0.048" rpy_caster="0 0 0" side="front_right"/>
-    <xacro:ota_swivel base_link="${base_link}" xyz_caster="0.37 0.22 -0.048" rpy_caster="0 0 0" side="front_left"/>
-    <xacro:ota_swivel base_link="${base_link}" xyz_caster="-0.37 -0.22 -0.048" rpy_caster="0 0 0" side="back_right"/>
-    <xacro:ota_swivel base_link="${base_link}" xyz_caster="-0.37 0.22 -0.048" rpy_caster="0 0 0" side="back_left"/>
+    <xacro:ota_swivel base_link="${base_link}" xyz_caster="0.37 -0.22 -0.048" rpy_caster="0 0 0" side="front_right" prefix="${prefix}"/>
+    <xacro:ota_swivel base_link="${base_link}" xyz_caster="0.37 0.22 -0.048" rpy_caster="0 0 0" side="front_left" prefix="${prefix}"/>
+    <xacro:ota_swivel base_link="${base_link}" xyz_caster="-0.37 -0.22 -0.048" rpy_caster="0 0 0" side="back_right" prefix="${prefix}"/>
+    <xacro:ota_swivel base_link="${base_link}" xyz_caster="-0.37 0.22 -0.048" rpy_caster="0 0 0" side="back_left" prefix="${prefix}"/>
     <!-- <xacro:ota_ir base_link="${base_link}" link_name="ota_ir" xyz_ir="0.503 0.0 0.175" rpy_ir="0 0 0"/>
     <xacro:ota_wheel base_link="${base_link}" xyz_hub="0 -0.305 0.10" rpy_hub="0 0 0" side="left"/>
@@ -44,5 +46,5 @@
     <xacro:ota_swivel base_link="${base_link}" xyz_caster="-0.37 0.217 0.12" rpy_caster="0 0 0" side="back_left"/> -->
     <!-- Differential Drive Plugin (AGV hareketi için) -->
-    <xacro:ota_diff_drive base_link="${base_link}"/>
+    <xacro:ota_diff_drive base_link="${base_link}" prefix="${prefix}"/>
     <!-- Joint State Publisher Plugin -->
     <xacro:ota_joints_state_publisher/>

File: mobile_manipulator_description/urdf/ota/ota_plugin.xacro (robot description, xacro)
@@ -11,11 +11,11 @@
   </xacro:macro>
   <!-- ✅ Differential Drive Plugin (Gazebo Harmonic: gz-sim-diff-drive-system) -->
-  <xacro:macro name="ota_diff_drive" params="base_link">
+  <xacro:macro name="ota_diff_drive" params="base_link prefix:=''">
     <gazebo>
       <plugin name="gz::sim::systems::DiffDrive"
               filename="gz-sim-diff-drive-system">
         <!-- Tekerlek eklemleri (ota_wheel.xacro'daki joint isimleri) -->
-        <left_joint>wheel_left_base</left_joint>
-        <right_joint>wheel_right_base</right_joint>
+        <left_joint>${prefix}wheel_left_base</left_joint>
+        <right_joint>${prefix}wheel_right_base</right_joint>
         <!-- Geometri -->
         <wheel_separation>0.60</wheel_separation>

File: mobile_manipulator_description/urdf/ota/ota_wheel.xacro (robot description, xacro)
@@ -1,7 +1,7 @@
 <?xml version="1.0"?>
 <robot xmlns:xacro="http://www.ros.org/wiki/xacro">
-  <xacro:macro name="ota_wheel" params="base_link xyz_hub rpy_hub side">
+  <xacro:macro name="ota_wheel" params="base_link xyz_hub rpy_hub side prefix:=''">
     <!-- === WHEEL VISUAL === -->
-    <link name="wheel_${side}_link">
+    <link name="${prefix}wheel_${side}_link">
       <visual>
         <origin xyz="0 0 0" rpy="0 0 1.570796"/>
@@ -29,12 +29,12 @@
     </link>
     <!-- === WHEEL JOINT === -->
-    <joint name="wheel_${side}_base" type="continuous">
+    <joint name="${prefix}wheel_${side}_base" type="continuous">
       <origin xyz="${xyz_hub}" rpy="${rpy_hub}"/>
       <parent link="${base_link}"/>
-      <child link="wheel_${side}_link"/>
+      <child link="${prefix}wheel_${side}_link"/>
       <axis xyz="0 1 0"/>
     </joint>
     <!-- Gazebo wheel parameters -->
-    <gazebo reference="wheel_${side}_link">
+    <gazebo reference="${prefix}wheel_${side}_link">
       <mu1>1.0</mu1>
       <mu2>1.0</mu2>
