Commit message: Kawasaki ros2_control

File: rs005l_description/urdf/rs005l.ros2_control.xacro (robot description, xacro)
@@ -8,4 +8,7 @@
     sim_ignition:=false
     fake_sensor_commands:=false
+    robot_ip:=192.168.3.7
+    robot_port:=11111
+    cmd_threshold_rad:=0.001
     ">
     <ros2_control name="${name}" type="system">
@@ -20,5 +23,30 @@
           <param name="calculate_dynamics">true</param>
         </xacro:if>
+        <!-- Real Kawasaki RS005L hardware via SIR TCP/IP protocol -->
+        <xacro:unless value="${sim_ignition or use_fake_hardware}">
+          <plugin>kawasaki_ros2_control/KawasakiHardwareInterface</plugin>
+          <param name="robot_ip">${robot_ip}</param>
+          <param name="robot_port">${robot_port}</param>
+          <param name="cmd_threshold_rad">${cmd_threshold_rad}</param>
+        </xacro:unless>
       </hardware>
+      <!-- AGV prismatic joint (world_to_agv):
+           - fake hardware → rs005l GenericSystem altında (7-DOF tek system)
+           - gerçek hardware → ota_system TopicBasedSystem altında
+             (KawasakiHardwareInterface sadece 6 eklem kabul eder) -->
+      <xacro:if value="${use_fake_hardware}">
+        <joint name="world_to_agv">
+          <command_interface name="position"/>
+          <command_interface name="velocity">
+            <param name="min">-1.25</param>
+            <param name="max">1.25</param>
+          </command_interface>
+          <state_interface name="position">
+              <param name="initial_value">1.0</param>
+          </state_interface>
+          <state_interface name="velocity"/>
+          <state_interface name="effort"/>
+        </joint>
+      </xacro:if>
       <!-- orjinalinde command interface effort bunu sormak lazım -->
       <joint name="${tf_prefix}joint1">
