Commit message: Ready for Use Case Developments

File: Universal_Robots_ROS2_Tutorials/my_robot_cell/my_robot_cell_control/urdf/whole_cell_real.urdf.xacro (robot description, xacro)
@@ -49,5 +49,5 @@
   <xacro:arg name="kawasaki_tf_prefix" default=""/>
   <!-- AGV pozisyonu (world frame'e göre) -->
-  <xacro:arg name="agv_x" default="-2.301949"/>
+  <xacro:arg name="agv_x" default="-2.301959"/>
   <xacro:arg name="agv_y" default="0.135135131"/>
   <xacro:arg name="agv_z" default="0.17"/>

File: Universal_Robots_ROS2_Tutorials/my_robot_cell/my_robot_cell_control/urdf/whole_cell_sim.urdf.xacro (robot description, xacro)
@@ -61,5 +61,5 @@
   <xacro:arg name="kawasaki_simulation_controllers" default=""/>
   <!-- AGV spawn pozisyonu (world frame'e göre) -->
-  <xacro:arg name="agv_x" default="-2.301949"/>
+  <xacro:arg name="agv_x" default="-2.301959"/>
   <xacro:arg name="agv_y" default="0.135135131"/>
   <xacro:arg name="agv_z" default="0.17"/>

File: Universal_Robots_ROS2_Tutorials/my_robot_cell/my_robot_cell_description/urdf/my_robot_cell_macro.xacro (robot description, xacro)
@@ -51,17 +51,21 @@
       <origin xyz="0 0 0" rpy="0 0 0"/>
     </xacro:chassis_assembly> -->
-    <!-- CHASSIS LINK - devre dışı bırakıldı, platform/door/door1 ile değiştirildi
     <link name="${tf_prefix}chassis">
       <inertial>
         <origin xyz="-1.124731 1.232845 1.108302" rpy="0 0 0"/>
         <mass value="120.90442642947052"/>
-        <inertia ixx="129.47263" ixy="-0.023527" ixz="-0.011644"
-                iyy="73.136591" iyz="-1.726202"
-                izz="85.878511"/>
-      </inertial>
-      <visual>
-        <origin xyz="0 0 0" rpy="0 0 0"/>
-        <geometry>
-          <mesh filename="file:////home/cem/colcon_ws/src/Universal_Robots_ROS2_Description/meshes/ur10e/collision/chassis.stl" scale="0.001 0.001 0.001"/>
+        <inertia
+            ixx="1.363e6"
+            ixy="-903.3"
+            ixz="1.847e4"
+            iyy="8.130e5"
+            iyz="-385.3"
+            izz="1.039e6"/>
+      </inertial>
+      <visual>
+        <origin xyz="0 0 0" rpy="0 0 0"/>
+        <geometry>
+          <mesh filename="file:////home/cem/colcon_ws/src/Universal_Robots_ROS2_Description/meshes/ur10e/collision/chassis.stl"
+                scale="0.001 0.001 0.001"/>
         </geometry>
         <material name="chassis_material">
@@ -72,11 +76,11 @@
         <origin xyz="0 0 0" rpy="0 0 0"/>
         <geometry>
-          <mesh filename="file:////home/cem/colcon_ws/src/Universal_Robots_ROS2_Description/meshes/ur10e/collision/chassis.stl" scale="0.001 0.001 0.001"/>
-        </geometry>
-      </collision>
-    </link>
-    -->
+          <mesh filename="file:////home/cem/colcon_ws/src/Universal_Robots_ROS2_Description/meshes/ur10e/collision/chassis.stl"
+                scale="0.001 0.001 0.001"/>
+        </geometry>
+      </collision>
+    </link>
     <!-- Platform - Bodies(1): mass=205.0 kg, inertia CAD'dan alındı -->
-    <link name="${tf_prefix}platform">
+    <!-- <link name="${tf_prefix}platform">
       <inertial>
         <origin xyz="-1.101122 1.387607 0.574201" rpy="0 0 0"/>
@@ -99,7 +103,7 @@
         </geometry>
       </collision>
-    </link>
+    </link> -->
     <!-- Door - araba kapısı (~18 kg, 1.1m x 0.9m x 0.05m çelik) -->
-    <link name="${tf_prefix}windowlessdoor">
+    <!-- <link name="${tf_prefix}windowlessdoor">
       <inertial>
         <origin xyz="-0.864306 0.816343 0.934094" rpy="0 0 0"/>
@@ -122,7 +126,7 @@
         </geometry>
       </collision>
-    </link>
+    </link> -->
     <!-- Door1 - araba kapısı (~18 kg, 1.1m x 0.9m x 0.05m çelik) -->
-    <link name="${tf_prefix}windowdoor">
+    <!-- <link name="${tf_prefix}windowdoor">
       <inertial>
         <origin xyz="-0.844038 1.994389 0.74421" rpy="0 0 0"/>
@@ -145,5 +149,5 @@
         </geometry>
       </collision>
-    </link>
+    </link> -->
     <link name="${tf_prefix}robot_mount">
       <inertial>
@@ -166,44 +170,4 @@
       </collision>
     </link>
-    <!-- <link name="${tf_prefix}wall_door">
-      <inertial>
-        <origin rpy="0 0 0" xyz="600.0 3235.0 550.0"/>
-        <mass value="8.04925448455695"/>
-        <inertia ixx="10.53" ixy="0.0" ixz="0.0" iyy="22.88" iyz="0.0" izz="12.52"/>
-      </inertial>
-      <visual>
-        <origin rpy="0 0 0" xyz="0 0 0"/>
-        <geometry>
-          <mesh filename="file:////home/cem/colcon_ws/src/Universal_Robots_ROS2_Description/meshes/ur10e/collision/wall_door.stl" scale="0.001 0.001 0.001"/>
-        </geometry>
-        <material name="silver"/>
-      </visual>
-      <collision>
-        <origin rpy="0 0 0" xyz="0 0 0"/>
-        <geometry>
-          <mesh filename="file:////home/cem/colcon_ws/src/Universal_Robots_ROS2_Description/meshes/ur10e/collision/wall_door.stl" scale="0.001 0.001 0.001"/>
-        </geometry>
-      </collision>
-    </link>
-    <link name="${tf_prefix}wall_server">
-      <inertial>
-        <origin rpy="0 0 0" xyz="-175.0 -1020.0 550.0"/>
-        <mass value="12.04925448455695"/>
-        <inertia ixx="24.14" ixy="0.0" ixz="0.0" iyy="17.36" iyz="0.0" izz="14.98"/>
-      </inertial>
-      <visual>
-        <origin rpy="0 0 0" xyz="0 0 0"/>
-        <geometry>
-          <mesh filename="file:////home/cem/colcon_ws/src/Universal_Robots_ROS2_Description/meshes/ur10e/collision/wall_server.stl" scale="0.001 0.001 0.001"/>
-        </geometry>
-        <material name="silver"/>
-      </visual>
-      <collision>
-        <origin rpy="0 0 0" xyz="0 0 0"/>
-        <geometry>
-          <mesh filename="file:////home/cem/colcon_ws/src/Universal_Robots_ROS2_Description/meshes/ur10e/collision/wall_server.stl" scale="0.001 0.001 0.001"/>
-        </geometry>
-      </collision>
-    </link> -->
     <link name="${tf_prefix}alumunium_table">
       <inertial>
@@ -329,5 +293,4 @@
       <dynamics damping="100.0" friction="50.0"/>
     </joint>
-    <!-- CHASSIS JOINT - devre dışı bırakıldı
     <joint name="${tf_prefix}base_to_chassis" type="fixed">
       <parent link="${parent}"/>
@@ -335,6 +298,5 @@
       <origin xyz="0 0 0" rpy="0 0 0"/>
     </joint>
-    -->
-    <joint name="${tf_prefix}base_to_platform" type="fixed">
+    <!-- <joint name="${tf_prefix}base_to_platform" type="fixed">
       <parent link="${parent}"/>
       <child link="${tf_prefix}platform"/>
@@ -350,5 +312,5 @@
       <child link="${tf_prefix}windowdoor"/>
       <origin xyz="0 0 0" rpy="0 0 0"/>
-    </joint>
+    </joint> -->
     <joint name="${tf_prefix}base_to_alumuniumtable" type="fixed">
       <parent link="${parent}"/>

File: Universal_Robots_ROS2_Tutorials/my_robot_cell/my_robot_cell_description/urdf/simrobot_my_robot_cell_macro.xacro (robot description, xacro)
@@ -43,17 +43,21 @@
     </xacro:chassis_assembly>
     -->
-    <!-- CHASSIS LINK - devre dışı bırakıldı
     <link name="${tf_prefix}chassis">
       <inertial>
         <origin xyz="-1.124731 1.232845 1.108302" rpy="0 0 0"/>
         <mass value="120.90442642947052"/>
-        <inertia ixx="129.47263" ixy="-0.023527" ixz="-0.011644"
-                iyy="73.136591" iyz="-1.726202"
-                izz="85.878511"/>
-      </inertial>
-      <visual>
-        <origin xyz="0 0 0" rpy="0 0 0"/>
-        <geometry>
-          <mesh filename="file:////home/cem/colcon_ws/src/Universal_Robots_ROS2_Description/meshes/ur10e/collision/chassis.stl" scale="0.001 0.001 0.001"/>
+        <inertia
+            ixx="1.363e6"
+            ixy="-903.3"
+            ixz="1.847e4"
+            iyy="8.130e5"
+            iyz="-385.3"
+            izz="1.039e6"/>
+      </inertial>
+      <visual>
+        <origin xyz="0 0 0" rpy="0 0 0"/>
+        <geometry>
+          <mesh filename="file:////home/cem/colcon_ws/src/Universal_Robots_ROS2_Description/meshes/ur10e/collision/chassis.stl"
+                scale="0.001 0.001 0.001"/>
         </geometry>
         <material name="chassis_material">
@@ -64,11 +68,11 @@
         <origin xyz="0 0 0" rpy="0 0 0"/>
         <geometry>
-          <mesh filename="file:////home/cem/colcon_ws/src/Universal_Robots_ROS2_Description/meshes/ur10e/collision/chassis.stl" scale="0.001 0.001 0.001"/>
-        </geometry>
-      </collision>
-    </link>
-    -->
+          <mesh filename="file:////home/cem/colcon_ws/src/Universal_Robots_ROS2_Description/meshes/ur10e/collision/chassis.stl"
+                scale="0.001 0.001 0.001"/>
+        </geometry>
+      </collision>
+    </link>
     <!-- Platform - Bodies(1): mass=205.0 kg, inertia CAD'dan alındı -->
-    <link name="${tf_prefix}platform">
+    <!-- <link name="${tf_prefix}platform">
       <inertial>
         <origin xyz="-1.101122 1.387607 0.574201" rpy="0 0 0"/>
@@ -91,7 +95,7 @@
         </geometry>
       </collision>
-    </link>
+    </link> -->
     <!-- Door - araba kapısı (~18 kg, 1.1m x 0.9m x 0.05m çelik) -->
-    <link name="${tf_prefix}windowlessdoor">
+    <!-- <link name="${tf_prefix}windowlessdoor">
       <inertial>
         <origin xyz="-0.864306 0.816343 0.934094" rpy="0 0 0"/>
@@ -114,7 +118,7 @@
         </geometry>
       </collision>
-    </link>
+    </link> -->
     <!-- Door1 - araba kapısı (~18 kg, 1.1m x 0.9m x 0.05m çelik) -->
-    <link name="${tf_prefix}windowdoor">
+    <!-- <link name="${tf_prefix}windowdoor">
       <inertial>
         <origin xyz="-0.844038 1.994389 0.74421" rpy="0 0 0"/>
@@ -137,5 +141,5 @@
         </geometry>
       </collision>
-    </link>
+    </link> -->
     <link name="${tf_prefix}robot_mount">
       <inertial>
@@ -244,5 +248,4 @@
       <child link="${tf_prefix}table" />
     </joint>
-    <!-- CHASSIS JOINT - devre dışı bırakıldı
     <joint name="${tf_prefix}base_to_chassis" type="fixed">
       <parent link="${parent}"/>
@@ -250,6 +253,5 @@
       <origin xyz="0 0 0" rpy="0 0 0"/>
     </joint>
-    -->
-    <joint name="${tf_prefix}base_to_platform" type="fixed">
+    <!-- <joint name="${tf_prefix}base_to_platform" type="fixed">
       <parent link="${parent}"/>
       <child link="${tf_prefix}platform"/>
@@ -265,5 +267,5 @@
       <child link="${tf_prefix}windowdoor"/>
       <origin xyz="0 0 0" rpy="0 0 0"/>
-    </joint>
+    </joint> -->
     <!-- Linear axis joint - bu joint'in tam tanımı burada olmalı -->
     <joint name="${tf_prefix}base_to_robot_mount" type="prismatic">

File: mobile_manipulator_description/urdf/ota/ota_base.xacro (robot description, xacro)
@@ -85,12 +85,13 @@
       </visual>
     </gazebo> -->
-    <!-- cem.sdf: ifarlab_ray model pose = "0 0 0 0 0 0" → world origin -->
+    <!-- ifarlab_ray (şase rayı): kabinete 0.0497m (-Y), şaseye 0.1m (+X) kaydırıldı -->
     <joint name="${prefix}ifarlab_ray_joint" type="fixed">
       <parent link="world"/>
       <child link="${prefix}ifarlab_ray_link"/>
-      <origin xyz="0 0 0" rpy="0 0 0"/>
+      <origin xyz="0.095 -0.0497 0" rpy="0 0 0"/>
     </joint>
-    <!-- AGV başlangıç konumu: cem.sdf spawn pozisyonundan okundu
-         x=-2.301949  y=0.135135131  z=0.17  yaw=1.570796 (90°)
+    <!-- AGV başlangıç konumu (ifarlab_ray_link frame'e göre, orijinal değerler).
+         Ray frame zaten +0.1 X, -0.0787 Y kaydırıldığından AGV net world
+         pozisyonu: x≈-2.202, y≈0.056, z=0.165
          axis 1 0 0 = joint frame local X = yaw 90° nedeniyle world +Y yönü
          Bu eksende AGV ileri/geri hareket eder (ray üzerinde kayar) -->
