Commit message: Whole IFARLAB URDF

File: Universal_Robots_ROS2_Tutorials/my_robot_cell/my_robot_cell_description/urdf/simrobot_my_robot_cell_macro.xacro (robot description, xacro)
@@ -87,5 +87,5 @@
     <link name="${tf_prefix}alumunium_table">
       <inertial>
-        <origin rpy="0 0 0" xyz="681.141 2464.643 737.851"/>
+        <origin rpy="0 0 0" xyz="0.681141 2.464643 0.737851"/>
         <mass value="20.04925448455695"/>
         <inertia ixx="130.9" ixy="0.04503" ixz="0.9303" iyy="70.758" iyz="-0.03313" izz="139.1"/>
@@ -107,7 +107,7 @@
     <link name="${tf_prefix}conveyor_belt">
       <inertial>
-        <origin rpy="0 0 0" xyz="736.828 104.977 664.295"/>
-        <mass value="15.04925448455695"/>
-        <inertia ixx="0.061984" ixy="-0.003503" ixz="0.001551" iyy="0.069314" iyz="0.000564" izz="0.125682"/>
+        <origin rpy="0 0 0" xyz="0.731215 0.101822 0.642664"/>
+        <mass value="27.036586"/>
+        <inertia ixx="4.104" ixy="-0.008305" ixz="-0.010260" iyy="2.304" iyz="0.064250" izz="2.392"/>
       </inertial>
       <visual>

File: mobile_manipulator_description/urdf/ota/inertia_tensors.urdf.xacro (robot description, xacro)
@@ -1,7 +1,7 @@
 <?xml version="1.0"?>
+  <!-- Thanks to Martin Guenther
+  see https://github.com/uos/uos_tools/blob/fuerte/uos_common_urdf/common.xacro and
+  see http://answers.gazebosim.org/question/4372/the-inertia-matrix-explained/ -->
 <robot xmlns:xacro="http://ros.org/wiki/xacro">
-  <!-- Plugin makrolarını dahil et (DiffDrive, JointStatePublisher) -->
-  <xacro:include filename="$(find mobile_manipulator_description)/urdf/ota/ota_plugin.xacro"/>
-  <!-- Inertia helper macros -->
   <property name="M_PI" value="3.1415926535897931" />
   <!-- see https://secure.wikimedia.org/wikipedia/en/wiki/List_of_moment_of_inertia_tensors -->
@@ -16,28 +16,10 @@
     </inertial>
   </xacro:macro>
-  <xacro:macro name="sphere_inertial_with_origin" params="radius mass *origin">
-    <inertial>
-      <mass value="${mass}" />
-      <insert_block name="origin" />
-      <inertia ixx="${0.4 * mass * radius * radius}" ixy="0.0" ixz="0.0"
-        iyy="${0.4 * mass * radius * radius}" iyz="0.0"
-        izz="${0.4 * mass * radius * radius}" />
-    </inertial>
-  </xacro:macro>
   <xacro:macro name="cylinder_inertial" params="radius length mass">
     <inertial>
       <mass value="${mass}" />
       <origin xyz="0 0 0" />
-      <inertia ixx="${(1/12.0) * mass * (3 * radius * radius + length * length)}" ixy="0.0" ixz="0.0"
-        iyy="${(1/12.0) * mass * (3 * radius * radius + length * length)}" iyz="0.0"
-        izz="${0.5 * mass * radius * radius}" />
-    </inertial>
-  </xacro:macro>
-  <xacro:macro name="cylinder_inertial_with_origin" params="radius length mass *origin">
-    <inertial>
-      <mass value="${mass}" />
-      <insert_block name="origin" />
-      <inertia ixx="${(1/12.0) * mass * (3 * radius * radius + length * length)}" ixy="0.0" ixz="0.0"
-        iyy="${(1/12.0) * mass * (3 * radius * radius + length * length)}" iyz="0.0"
+      <inertia ixx="${0.0833333 * mass * (3 * radius * radius + length * length)}" ixy="0.0" ixz="0.0"
+        iyy="${0.0833333 * mass * (3 * radius * radius + length * length)}" iyz="0.0"
         izz="${0.5 * mass * radius * radius}" />
     </inertial>
@@ -52,4 +34,23 @@
     </inertial>
   </xacro:macro>
+  <!-- #################### versions with origin #################### -->
+  <xacro:macro name="sphere_inertial_with_origin" params="radius mass *origin">
+    <inertial>
+      <mass value="${mass}" />
+      <insert_block name="origin" />
+      <inertia ixx="${0.4 * mass * radius * radius}" ixy="0.0" ixz="0.0"
+        iyy="${0.4 * mass * radius * radius}" iyz="0.0"
+        izz="${0.4 * mass * radius * radius}" />
+    </inertial>
+  </xacro:macro>
+  <xacro:macro name="cylinder_inertial_with_origin" params="radius length mass *origin">
+    <inertial>
+      <mass value="${mass}" />
+      <insert_block name="origin" />
+      <inertia ixx="${0.0833333 * mass * (3 * radius * radius + length * length)}" ixy="0.0" ixz="0.0"
+        iyy="${0.0833333 * mass * (3 * radius * radius + length * length)}" iyz="0.0"
+        izz="${0.5 * mass * radius * radius}" />
+    </inertial>
+  </xacro:macro>
   <xacro:macro name="box_inertial_with_origin" params="x y z mass *origin">
     <inertial>

File: mobile_manipulator_description/urdf/ota/ota_base.xacro (robot description, xacro)
@@ -5,5 +5,5 @@
       <origin xyz="0 0 0" rpy=" 0 0 0"/>
       <visual>
-        <origin xyz="-0.1 0 -0.1625" rpy=" 0 0 0"/>
+        <origin xyz="0 0 -0.1625" rpy=" 0 0 0"/>
         <geometry>
           <mesh filename="file:////home/cem/colcon_ws/src/mobile_manipulator_description/meshes/ota/OTA-v0.7.stl" scale="0.001 0.001 0.001"/>

File: mobile_manipulator_description/urdf/ota/ota_caster.xacro (robot description, xacro)
@@ -18,5 +18,12 @@
         </geometry>
       </collision>
-      <xacro:cylinder_inertial radius="0.005" length="0.07" mass="1" />
+      <!-- <xacro:cylinder_inertial radius="0.005" length="0.07" mass="1"/> ORJİNALİ BÖYLE-->
+      <inertial>
+        <mass value="1" />
+        <origin xyz="0 0 0" rpy="0 0 0"/>
+        <inertia ixx="${0.0833333 * 1 * (3 * 0.005 * 0.005 + 0.07 * 0.07)}" ixy="0.0" ixz="0.0"
+          iyy="${0.0833333 * 1 * (3 * 0.005 * 0.005 + 0.07 * 0.07)}" iyz="0.0"
+          izz="${0.5 * 1 * 0.005 * 0.005}" />
+      </inertial>
     </link>
     <joint name="caster_${side}_joint" type="fixed">
@@ -41,5 +48,5 @@
       </visual>
     </gazebo>
-    <!-- <link name='caster_wheel_${side}_link'>
+    <link name='caster_wheel_${side}_link'>
       <visual>
         <origin xyz="0 0 0"/>
@@ -54,5 +61,12 @@
         </geometry>
       </collision>
-      <xacro:cylinder_inertial radius="0.042" length="0.02" mass="0.1" />
+      <!-- <xacro:cylinder_inertial radius="0.042" length="0.02" mass="0.1" /> ORJİNALİ BÖYLE -->
+      <inertial>
+        <mass value="0.1" />
+        <origin xyz="0 0 0" rpy="0 0 0"/>
+        <inertia ixx="${0.0833333 * 0.1 * (3 * 0.042 * 0.042 + 0.02 * 0.02)}" ixy="0.0" ixz="0.0"
+          iyy="${0.0833333 * 0.1 * (3 * 0.042 * 0.042 + 0.02 * 0.02)}" iyz="0.0"
+          izz="${0.5 * 0.1 * 0.042 * 0.042}" />
+      </inertial>
     </link>
     <joint name="caster_${side}_wheel_joint" type="fixed">
@@ -61,5 +75,5 @@
       <parent link="caster_${side}_link"/>
       <child link="caster_wheel_${side}_link"/>
-    </joint>   -->
+    </joint>
   </xacro:macro>
 </robot>

File: mobile_manipulator_description/urdf/ota/ota_wheel.xacro (robot description, xacro)
@@ -19,5 +19,12 @@
       </collision>
       <!-- === WHEEL INERTIA === -->
-      <xacro:cylinder_inertial radius="0.102" length="0.02" mass="5"/>
+      <!-- <xacro:cylinder_inertial radius="0.102" length="0.02" mass="5"/>ORJİNALİ BÖYLE -->
+      <inertial>
+        <mass value="5" />
+        <origin xyz="0 0 0" rpy="0 0 0"/>
+        <inertia ixx="${0.0833333 * 5 * (3 * 0.102 * 0.102 + 0.02 * 0.02)}" ixy="0.0" ixz="0.0"
+          iyy="${0.0833333 * 5 * (3 * 0.102 * 0.102 + 0.02 * 0.02)}" iyz="0.0"
+          izz="${0.5 * 5 * 0.102 * 0.102}" />
+      </inertial>
     </link>
     <!-- === WHEEL JOINT === -->
