Commit message: MultiRobot Chassis Inspection

File: Universal_Robots_ROS2_Tutorials/my_robot_cell/my_robot_cell_description/urdf/my_robot_cell_macro.xacro (robot description, xacro)
@@ -46,5 +46,32 @@
         </geometry>
       </collision>
-    </link>
+      <!-- LINEAR-AXIS MOTOR HOUSING, enlarged 2026-09-08.
+           base_link.stl already carries this protrusion as 12 triangles spanning
+           x -0.492..-0.317, y 0.040..0.120, z 0.492..0.597 (0.175 x 0.080 x 0.105 m)
+           at the y=0 end of the rail, and a UR joint struck the real housing there, so
+           the modelled volume was too small. This box supersedes it: 0.20 m out
+           along -X, 0.15 m wide grown toward -Y, 0.14 m tall. The BACK face
+           (x=-0.317, where it meets the rail body) and the +Y face (y=0.120) are
+           unchanged; the box grows forward along -X, toward -Y, and SYMMETRICALLY in
+           height: 1.75 cm up and 1.75 cm down, so z runs 0.4745..0.6145 around the
+           original feature's own centre. Growing upward past the rail top (z=0.597)
+           is safe even though ur10e_robot_mount rides this rail from z=0.583 up:
+           the mount's collision mesh starts at x=-0.310 and this box ends at
+           x=-0.317, so the two never meet at any rail position.
+           The mesh feature stays where it is, fully inside this box. -->
+      <collision>
+        <origin rpy="0 0 0" xyz="-0.417 0.045 0.5445"/>
+        <geometry>
+          <box size="0.20 0.15 0.14"/>
+        </geometry>
+      </collision>
+      <visual>
+        <origin rpy="0 0 0" xyz="-0.417 0.045 0.5445"/>
+        <geometry>
+          <box size="0.20 0.15 0.14"/>
+        </geometry>
+        <material name="silver"/>
+      </visual>
+</link>
     <!-- Chassis assembly - tüm PART1-PART44 parçalarını içerir -->
     <xacro:chassis_assembly tf_prefix="${tf_prefix}" parent="${parent}">

File: Universal_Robots_ROS2_Tutorials/my_robot_cell/my_robot_cell_description/urdf/simrobot_my_robot_cell_macro.xacro (robot description, xacro)
@@ -37,5 +37,32 @@
         </geometry>
       </collision>
-    </link>
+      <!-- LINEAR-AXIS MOTOR HOUSING, enlarged 2026-09-08.
+           base_link.stl already carries this protrusion as 12 triangles spanning
+           x -0.492..-0.317, y 0.040..0.120, z 0.492..0.597 (0.175 x 0.080 x 0.105 m)
+           at the y=0 end of the rail, and a UR joint struck the real housing there, so
+           the modelled volume was too small. This box supersedes it: 0.20 m out
+           along -X, 0.15 m wide grown toward -Y, 0.14 m tall. The BACK face
+           (x=-0.317, where it meets the rail body) and the +Y face (y=0.120) are
+           unchanged; the box grows forward along -X, toward -Y, and SYMMETRICALLY in
+           height: 1.75 cm up and 1.75 cm down, so z runs 0.4745..0.6145 around the
+           original feature's own centre. Growing upward past the rail top (z=0.597)
+           is safe even though ur10e_robot_mount rides this rail from z=0.583 up:
+           the mount's collision mesh starts at x=-0.310 and this box ends at
+           x=-0.317, so the two never meet at any rail position.
+           The mesh feature stays where it is, fully inside this box. -->
+      <collision>
+        <origin rpy="0 0 0" xyz="-0.417 0.045 0.5445"/>
+        <geometry>
+          <box size="0.20 0.15 0.14"/>
+        </geometry>
+      </collision>
+      <visual>
+        <origin rpy="0 0 0" xyz="-0.417 0.045 0.5445"/>
+        <geometry>
+          <box size="0.20 0.15 0.14"/>
+        </geometry>
+        <material name="silver"/>
+      </visual>
+</link>
     <xacro:chassis_assembly tf_prefix="${tf_prefix}" parent="${parent}">
       <origin xyz="0 0 0" rpy="0 0 0"/>

Commit message: Bug fix

File: Universal_Robots_ROS2_Tutorials/my_robot_cell/my_robot_cell_description/urdf/my_robot_cell_macro.xacro (robot description, xacro)
@@ -71,5 +71,43 @@
           <box size="0.20 0.15 0.14"/>
         </geometry>
-        <material name="silver"/>
+        <material name="table_blocks_grey"><color rgba="0.7 0.7 0.7 1.0"/></material>
+      </visual>
+      <!-- CABLE CHANNEL on the chassis-facing side of the linear axis, raised
+           2026-09-11. base_link.stl carries it as two blocks, x -0.317..-0.237 and
+           z 0.447..0.597, split at y 0.975 / 1.055 (y 0.040..0.975 and 1.055..2.405).
+           The real channel stands about 5 cm taller than that, so these two boxes
+           supersede the mesh blocks with the top at z=0.647, same footprint, same y
+           split. 5 cm is close to the limit: the carriage (ur10e_robot_mount) has a
+           bracket directly above this footprint whose lowest point is z=0.6524, so the
+           gap left is ~5 mm. Going above 0.652 would put the model INSIDE the
+           carriage, and MoveIt would never say so: ur10e_table <-> ur10e_robot_mount,
+           base_link_inertia and shoulder_link are all disabled in the SRDF.
+           Recorded UR trajectories pass right at the padded clearance above these
+           blocks, so after this change they must be re-recorded (force_replan). -->
+      <collision>
+        <origin rpy="0 0 0" xyz="-0.277 0.5075 0.547"/>
+        <geometry>
+          <box size="0.080 0.935 0.200"/>
+        </geometry>
+      </collision>
+      <collision>
+        <origin rpy="0 0 0" xyz="-0.277 1.730 0.547"/>
+        <geometry>
+          <box size="0.080 1.350 0.200"/>
+        </geometry>
+      </collision>
+      <visual>
+        <origin rpy="0 0 0" xyz="-0.277 0.5075 0.547"/>
+        <geometry>
+          <box size="0.080 0.935 0.200"/>
+        </geometry>
+        <material name="table_blocks_grey"><color rgba="0.7 0.7 0.7 1.0"/></material>
+      </visual>
+      <visual>
+        <origin rpy="0 0 0" xyz="-0.277 1.730 0.547"/>
+        <geometry>
+          <box size="0.080 1.350 0.200"/>
+        </geometry>
+        <material name="table_blocks_grey"><color rgba="0.7 0.7 0.7 1.0"/></material>
       </visual>
 </link>

File: Universal_Robots_ROS2_Tutorials/my_robot_cell/my_robot_cell_description/urdf/simrobot_my_robot_cell_macro.xacro (robot description, xacro)
@@ -62,5 +62,43 @@
           <box size="0.20 0.15 0.14"/>
         </geometry>
-        <material name="silver"/>
+        <material name="sim_table_blocks_grey"><color rgba="0.8 0.8 0.8 1.0"/></material>
+      </visual>
+      <!-- CABLE CHANNEL on the chassis-facing side of the linear axis, raised
+           2026-09-11. base_link.stl carries it as two blocks, x -0.317..-0.237 and
+           z 0.447..0.597, split at y 0.975 / 1.055 (y 0.040..0.975 and 1.055..2.405).
+           The real channel stands about 5 cm taller than that, so these two boxes
+           supersede the mesh blocks with the top at z=0.647, same footprint, same y
+           split. 5 cm is close to the limit: the carriage (ur10e_robot_mount) has a
+           bracket directly above this footprint whose lowest point is z=0.6524, so the
+           gap left is ~5 mm. Going above 0.652 would put the model INSIDE the
+           carriage, and MoveIt would never say so: ur10e_table <-> ur10e_robot_mount,
+           base_link_inertia and shoulder_link are all disabled in the SRDF.
+           Recorded UR trajectories pass right at the padded clearance above these
+           blocks, so after this change they must be re-recorded (force_replan). -->
+      <collision>
+        <origin rpy="0 0 0" xyz="-0.277 0.5075 0.547"/>
+        <geometry>
+          <box size="0.080 0.935 0.200"/>
+        </geometry>
+      </collision>
+      <collision>
+        <origin rpy="0 0 0" xyz="-0.277 1.730 0.547"/>
+        <geometry>
+          <box size="0.080 1.350 0.200"/>
+        </geometry>
+      </collision>
+      <visual>
+        <origin rpy="0 0 0" xyz="-0.277 0.5075 0.547"/>
+        <geometry>
+          <box size="0.080 0.935 0.200"/>
+        </geometry>
+        <material name="sim_table_blocks_grey"><color rgba="0.8 0.8 0.8 1.0"/></material>
+      </visual>
+      <visual>
+        <origin rpy="0 0 0" xyz="-0.277 1.730 0.547"/>
+        <geometry>
+          <box size="0.080 1.350 0.200"/>
+        </geometry>
+        <material name="sim_table_blocks_grey"><color rgba="0.8 0.8 0.8 1.0"/></material>
       </visual>
 </link>
