Commit message: Multi-Robot Inspection

File: Universal_Robots_ROS2_Description/urdf/ur_macro.xacro (robot description, xacro)
@@ -585,4 +585,18 @@
       <child link="${tf_prefix}rgb_optical_frame"/>
     </joint>
+    <!-- Gerçek SICK Visionary-T Mini optik frame'i (Kawasaki'nin
+         kawasaki_sick_optical_frame karşılığı). depth_optical_frame IK/plan için
+         kullanılır; gerçek SICK bulutu ona göre görüş ekseni etrafında ~60° dönük
+         gelir, o yüzden gerçek bulut IK frame'ini bozmadan BU kalibre frame'e
+         damgalanır. RViz'de (Fixed Frame=world) bulut şaseye oturana kadar
+         ur_cloud_calibrator ile ayarlandı: xyz 0 0 -0.01, rpy 0 0 1.04720 (=60° yaw).
+         Gerçek UR SICK node frame_id + pointcloud_transformer_ur target_frame +
+         executor real_ur_sensor_frame hepsi bu frame'e işaret eder. -->
+    <joint name="${tf_prefix}ur_sick_optical_joint" type="fixed">
+      <origin xyz="0 0 -0.01" rpy="0 0 1.04720"/>
+      <parent link="${tf_prefix}depth_optical_frame"/>
+      <child link="${tf_prefix}sick_optical_frame"/>
+    </joint>
+    <link name="${tf_prefix}sick_optical_frame"/>
     <xacro:arg name="use_gripper" default="$(optenv ENV_USE_GRIPPER false)"/>
     <xacro:arg name="use_fake_hardware" default="$(optenv ENV_USE_FAKE_HARDWARE false)"/>

File: mobile_manipulator_description/urdf/khi_rs/rs005l_macro.xacro (robot description, xacro)
@@ -309,4 +309,16 @@
     </joint>
     <link name="${tf_prefix}camera_rgb_optic_frame"/>
+    <!-- Gerçek SICK Visionary-T Mini optik frame'i. camera_rgb_optic_frame Gazebo
+         sim kamerası için oryante edilmiştir (<gazebo reference=camera_rgb_optic_frame>);
+         gerçek SICK bulutu optik konvansiyon farkı nedeniyle ona göre dönüktür.
+         RViz'de (Fixed Frame=world) bulut şaseye oturana kadar kalibre edildi:
+         rpy = -pi/2, -pi/2, -pi/2 (konum ofseti gerekmedi). Gerçek bulut bu frame'e
+         damgalanır (sick_kawasaki node frame_id + pointcloud_transformer target). -->
+    <joint name="${tf_prefix}kawasaki_sick_optical_joint" type="fixed">
+       <origin xyz="-0.02 0 0" rpy="-1.5708 -1.5708 -1.5708"/>
+       <parent link="${tf_prefix}camera_rgb_optic_frame"/>
+       <child link="${tf_prefix}kawasaki_sick_optical_frame"/>
+    </joint>
+    <link name="${tf_prefix}kawasaki_sick_optical_frame"/>
     <xacro:if value="${sim_ignition}">
       <!-- NOT: gz-sim-sensors-system plugin'i world SDF'de (ifarlab.sdf) zaten

Commit message: GR+TrajOpt

File: Universal_Robots_ROS2_Description/urdf/ur_macro.xacro (robot description, xacro)
@@ -628,7 +628,33 @@
          ur_cloud_calibrator ile ayarlandı: xyz 0 0 -0.01, rpy 0 0 1.04720 (=60° yaw).
          Gerçek UR SICK node frame_id + pointcloud_transformer_ur target_frame +
-         executor real_ur_sensor_frame hepsi bu frame'e işaret eder. -->
+         executor real_ur_sensor_frame hepsi bu frame'e işaret eder.
+         Z DÜZELTMESİ -0.01 -> +0.035 (14 Ağu 2026).
+         Belirti: kol konveyördeki kutunun ~4 cm üstünde kalıyordu.
+         Sapma MESH'E DEĞİL, ŞERİT METREYE karşı ölçüldü. Mesh'e karşı
+         doğrulama bugün iki kez yanılttı, çünkü conveyorbelt.stl gerçek
+         konveyörü temsil etmiyor (yan korkuluk yüksekliği tutmuyor).
+         Ölçüm zinciri:
+           kap ağzı, kol TOUCH pozundayken   TF 0.9995 / metre 1.00-1.01
+             -> TF dogru, kol zinciri saglam, dunya z=0 = yer
+           kap ile kutunun ustu arasi bosluk  0.040 (gozle)
+           kutu yuksekligi                    0.114 (metre)
+             -> gercek bant = 1.000 - 0.040 - 0.114 = 0.845
+           metreyle dogrudan bant             0.845  (birebir tuttu)
+         Algının okudukları:
+           bant duzlemi        0.8900  (42580 nokta, std 1.92 mm)  -> +45.0 mm
+           kutunun ustu/temas  1.005   (gercek 0.960)              -> +45.0 mm
+         Iki bagimsiz yuzeyde ayni sapma: duzgun bir otelemedir.
+         Bu origin PARENT (depth_optical_frame) Z ekseni boyuncadır, dünya
+         Z'si boyunca değil. Bu pozda optik eksen dünyada [-0.002 0.002
+         -1.000], dikeyden 0.2 derece sapık, cos = -1.0000:
+             d = -(+0.0450) / -1.0000 = +0.0450
+             -0.01 + 0.045 = +0.035
+         Kamera neredeyse tam dik baktigi icin duzeltme birebir cikti.
+         NOT: aynı gün base_to_conveyorbelt de -0.0068'e alındı. O, MoveIt'in
+         çarpışma modelini gerçek banda oturtur; buradaki 45 mm ise kolun
+         nereye gittiğini belirleyen algı hatasıdır. İkisi ayrı şeylerdir ve
+         birbirinin yerine geçmez. -->
     <joint name="${tf_prefix}ur_sick_optical_joint" type="fixed">
-      <origin xyz="0 0 -0.01" rpy="0 0 1.04720"/>
+      <origin xyz="0 0 0.035" rpy="0 0 1.04720"/>
       <parent link="${tf_prefix}depth_optical_frame"/>
       <child link="${tf_prefix}sick_optical_frame"/>

File: Universal_Robots_ROS2_Tutorials/my_robot_cell/my_robot_cell_description/urdf/my_robot_cell_macro.xacro (robot description, xacro)
@@ -48,7 +48,7 @@
     </link>
     <!-- Chassis assembly - tüm PART1-PART44 parçalarını içerir -->
-    <!-- <xacro:chassis_assembly tf_prefix="${tf_prefix}" parent="${parent}">
-      <origin xyz="0 0 0" rpy="0 0 0"/>
-    </xacro:chassis_assembly> -->
+    <xacro:chassis_assembly tf_prefix="${tf_prefix}" parent="${parent}">
+      <origin xyz="0 0 0" rpy="0 0 0"/>
+    </xacro:chassis_assembly>
     <!-- <link name="${tf_prefix}chassis">
       <inertial>
@@ -81,5 +81,5 @@
       </collision>
     </link> -->
-    <link name="${tf_prefix}platform">
+    <!-- <link name="${tf_prefix}platform">
       <inertial>
         <origin xyz="-1.101122 1.387607 0.574201" rpy="0 0 0"/>
@@ -146,5 +146,5 @@
         </geometry>
       </collision>
-    </link>
+    </link> -->
     <link name="${tf_prefix}robot_mount">
       <inertial>
@@ -246,4 +246,36 @@
         <geometry>
           <mesh filename="file:////home/cem/colcon_ws/src/Universal_Robots_ROS2_Description/meshes/ur10e/collision/conveyorbelt.stl" scale="0.001 0.001 0.001"/>
+        </geometry>
+      </collision>
+      <!-- GERÇEK YAN KORKULUKLAR (14 Ağu 2026, bir çarpışmadan sonra eklendi).
+           conveyorbelt.stl korkulukları bandın sadece 3.1 mm üstünde bitiriyor
+           (link z 0.8549). GERÇEKTE korkulukların üstü yerden 0.900 m, yani
+           bandın (0.845) 55 mm üstünde. Model 52 mm alçak gösterdiği için
+           MoveIt korkulukları görmüyordu ve kol onlara çarptı.
+           Bu kutular mesh'in bıraktığı boşluğu dolduruyor: bandın üstünden
+           (link z 0.8518 = dünya 0.845) korkuluk üstüne (link z 0.9068 =
+           dünya 0.900) kadar, yükseklik 0.055.
+           Ayak izi mesh'ten ölçüldü (yukarı bakan yüzeyler, link z 0.8549):
+             sol  x 0.4903..0.5187   y -0.3824..0.4176
+             sağ  x 0.7803..0.8087   y -0.3824..0.5176
+           Profil genişliği iki tarafta da 28.4 mm.
+           Link frame ile dünya arasında 6.8 mm var (base_to_conveyorbelt
+           origin z = -0.0068); buradaki bütün z'ler LINK frame'inde.
+           SADECE collision, visual YOK: bunlar mesh'in eksiğini kapatan
+           çarpışma hacimleri, ayrı bir fiziksel parça değil; RViz'de mesh'in
+           üstüne binen kutular olarak görünmeleri kafa karıştırır.
+           Ayrı bir link değil, conveyor_belt'in parçası: SRDF'teki mevcut
+           çarpışma çiftleri (upper_arm, forearm, wrist_*, suction_cup
+           denetleniyor) olduğu gibi geçerli kalsın diye. -->
+      <collision>
+        <origin rpy="0 0 0" xyz="0.5045 0.0176 0.8793"/>
+        <geometry>
+          <box size="0.0284 0.8000 0.0550"/>
+        </geometry>
+      </collision>
+      <collision>
+        <origin rpy="0 0 0" xyz="0.7945 0.0676 0.8793"/>
+        <geometry>
+          <box size="0.0284 0.9000 0.0550"/>
         </geometry>
       </collision>
@@ -295,5 +327,5 @@
       <origin xyz="0 0 0" rpy="0 0 0"/>
     </joint> -->
-    <joint name="${tf_prefix}base_to_platform" type="fixed">
+    <!-- <joint name="${tf_prefix}base_to_platform" type="fixed">
       <parent link="${parent}"/>
       <child link="${tf_prefix}platform"/>
@@ -309,5 +341,5 @@
       <child link="${tf_prefix}windowdoor"/>
       <origin xyz="0 0 0" rpy="0 0 0"/>
-    </joint>
+    </joint> -->
     <joint name="${tf_prefix}base_to_alumuniumtable" type="fixed">
       <parent link="${parent}"/>
@@ -325,8 +357,29 @@
       <origin xyz="0 0 0" rpy="0 0 0"/>
     </joint>
+    <!-- Konveyör yüksekliği (14 Ağu 2026, ŞERİT METREYLE doğrulandı).
+         Hizalama BANT YÜZEYİNE göre yapılır: kavrama da çarpışma da orada olur.
+         Mesh'in bant yüzeyi (üstten görünen yüzey, 5 mm ızgarayla ölçüldü;
+         bandın ortasında x 0.56..0.745, y -0.30..0.40 tamamen düz) bu joint
+         sıfırken z = 0.8518'de. Gerçek bant yerden 0.845 m.
+             0.845 - 0.8518 = -0.0068
+         Dünya z=0'ın yer olduğu bağımsız doğrulandı: kol TOUCH pozundayken
+         TF kap ağzını 0.9995'te gösterdi, yerden şerit metre 1.00-1.01 m.
+         MESH GERÇEK KONVEYÖRÜ TAM TEMSİL ETMİYOR, dikkat:
+           - Mesh'te yan raylar bandın 3.1 mm üstünde (z 0.8549 ham).
+             GERÇEKTE raylar yerden 0.900, yani bandın 55 mm üstünde.
+             Model bu korkulukları 52 mm alçak gösteriyor; MoveIt gerçek
+             korkulukları GÖRMÜYOR. Kol banda yandan yaklaşırsa çarpabilir.
+             Kalıcı çözüm: korkulukları ayrı bir çarpışma kutusu olarak ekle.
+           - Mesh'in altı bu haliyle z = -0.0318'e iniyor (yerin altı). Sadece
+             görsel; alt şase de gerçekle birebir değil.
+         TARİHÇE: bu değer bir ara +0.0451 yapıldı, çünkü hizalama YAN RAY
+         ölçümünden (0.900) türetilmişti ve mesh'in ray-bant mesafesinin
+         gerçeği yansıttığı varsayılmıştı. Yansıtmıyor: ray hizalandı ama
+         bant 51 mm yukarı çıktı, nokta bulutu konveyörün içine gömülmüş
+         göründü ve suction_cup ile conveyor_belt çarpışmaya başladı. -->
     <joint name="${tf_prefix}base_to_conveyorbelt" type="fixed">
       <parent link="${parent}"/>
       <child link="${tf_prefix}conveyor_belt"/>
-      <origin xyz="0 0 0" rpy="0 0 0"/>
+      <origin xyz="0 0 -0.0068" rpy="0 0 0"/>
     </joint>
     <joint name="${tf_prefix}bin_fixed" type="fixed">

File: Universal_Robots_ROS2_Tutorials/my_robot_cell/my_robot_cell_description/urdf/simrobot_my_robot_cell_macro.xacro (robot description, xacro)
@@ -38,7 +38,7 @@
       </collision>
     </link>
-    <!-- <xacro:chassis_assembly tf_prefix="${tf_prefix}" parent="${parent}">
-      <origin xyz="0 0 0" rpy="0 0 0"/>
-    </xacro:chassis_assembly> -->
+    <xacro:chassis_assembly tf_prefix="${tf_prefix}" parent="${parent}">
+      <origin xyz="0 0 0" rpy="0 0 0"/>
+    </xacro:chassis_assembly>
     <!-- <link name="${tf_prefix}chassis">
       <inertial>
@@ -71,5 +71,5 @@
       </collision>
     </link> -->
-    <link name="${tf_prefix}platform">
+    <!-- <link name="${tf_prefix}platform">
       <inertial>
         <origin xyz="-1.101122 1.387607 0.574201" rpy="0 0 0"/>
@@ -136,5 +136,5 @@
         </geometry>
       </collision>
-    </link>
+    </link> -->
     <link name="${tf_prefix}robot_mount">
       <inertial>
@@ -248,5 +248,5 @@
       <origin xyz="0 0 0" rpy="0 0 0"/>
     </joint> -->
-    <joint name="${tf_prefix}base_to_platform" type="fixed">
+    <!-- <joint name="${tf_prefix}base_to_platform" type="fixed">
       <parent link="${parent}"/>
       <child link="${tf_prefix}platform"/>
@@ -262,5 +262,5 @@
       <child link="${tf_prefix}windowdoor"/>
       <origin xyz="0 0 0" rpy="0 0 0"/>
-    </joint>
+    </joint> -->
     <!-- Linear axis joint - bu joint'in tam tanımı burada olmalı -->
     <joint name="${tf_prefix}base_to_robot_mount" type="prismatic">
