Commit message: Gazebo Harmonic+Stream

File: Universal_Robots_ROS2_Description/urdf/simrobot_ur.ros2_control.xacro (robot description, xacro)
@@ -22,4 +22,5 @@
     keep_alive_count:=2
     use_gripper:=false
+    use_vacuum_gripper:=false
     ">
     <ros2_control name="${name}" type="system">

File: Universal_Robots_ROS2_Description/urdf/simrobot_ur_macro.xacro (robot description, xacro)
@@ -85,5 +85,6 @@
     non_blocking_read:=true
     keep_alive_count:=2
-    use_gripper:=false"
+    use_gripper:=false
+    use_vacuum_gripper:=false"
     >
     <!-- Load configuration data from the provided .yaml files -->
@@ -129,4 +130,5 @@
         keep_alive_count="${keep_alive_count}"
         use_gripper="${use_gripper}"
+        use_vacuum_gripper="${use_vacuum_gripper}"
         />
     </xacro:if>
@@ -607,5 +609,5 @@
         <limit upper="0.001" lower="-0.026" effort="1000" velocity="10"/>
       </joint>
-      <link name="${tf_prefix}IMX_Camera">
+      <!-- <link name="${tf_prefix}IMX_Camera">
         <inertial>
           <origin xyz="-3.465374807465338e-05 0.0003801084631929186 0.006566275485619721" rpy="0 0 0"/>
@@ -626,6 +628,6 @@
           </geometry>
         </collision>
-      </link>
-      <joint name="${tf_prefix}IMX_Camera_joint" type="fixed">
+      </link> -->
+      <!-- <joint name="${tf_prefix}IMX_Camera_joint" type="fixed">
         <origin xyz="-0.058785 -0.012133 0.033972" rpy="0 0 0"/>
         <parent link="${tf_prefix}sick_camera"/>
@@ -634,5 +636,4 @@
       <link name="${tf_prefix}IMX_Camera_frame_link"/>
       <joint name="${tf_prefix}IMX_Camera_frame_joint" type="fixed">
-        <!-- Datasheet: toplam derinlik 24.68mm, optik merkez lensin önünde -->
         <origin xyz="0.0 0.025 0.0" rpy="0 0 0" />
         <parent link="${tf_prefix}IMX_Camera" />
@@ -641,5 +642,4 @@
       <gazebo reference="${tf_prefix}IMX_Camera_frame_link">
         <sensor name="${tf_prefix}imx179_camera" type="camera">
-          <!-- +Z yönüne bak (roll=-π/2) -->
           <pose>0 0 0 0 -1.5708 0</pose>
           <always_on>true</always_on>
@@ -647,5 +647,4 @@
           <visualize>false</visualize>
           <camera name="${tf_prefix}imx179_rgb">
-            <!-- 145 deg = 2.5307 rad -->
             <horizontal_fov>2.5307</horizontal_fov>
             <image>
@@ -660,5 +659,5 @@
           </camera>
         </sensor>
-      </gazebo>
+      </gazebo> -->
     </xacro:if>
     <link name="${tf_prefix}cable_channel_flange">
@@ -771,4 +770,57 @@
       <!-- IMX179 RGB camera (IMX_Camera linkine bağlı) -->
     </xacro:if>
+    <xacro:arg name="use_vacuum_gripper" default="$(optenv ENV_USE_VACUUM_GRIPPER false)"/>
+    <xacro:if value="$(arg use_vacuum_gripper)">
+      <link name="${tf_prefix}vacuum_gripper">
+        <inertial>
+          <origin xyz="0.03840935181996907 0.02553282574514726 0.01947430811837292" rpy="0 0 0"/>
+          <mass value="5.206908838469105"/>
+          <inertia ixx="0.007119" iyy="0.00672" izz="0.006537" ixy="0.000313" iyz="1e-06" ixz="-1e-06"/>
+        </inertial>
+        <visual>
+          <origin xyz="-1.120802 -0.533941 -0.69825" rpy="0 0 0"/>
+          <geometry>
+            <mesh filename="file:////home/cem/colcon_ws/src/Universal_Robots_ROS2_Description/meshes/ur10e/secondrobotcollision/vacuum_gripper.stl" scale="0.001 0.001 0.001"/>
+          </geometry>
+          <material name="silver"/>
+        </visual>
+        <collision>
+          <origin xyz="-1.120802 -0.533941 -0.69825" rpy="0 0 0"/>
+          <geometry>
+            <mesh filename="file:////home/cem/colcon_ws/src/Universal_Robots_ROS2_Description/meshes/ur10e/secondrobotcollision/vacuum_gripper.stl" scale="0.001 0.001 0.001"/>
+          </geometry>
+        </collision>
+      </link>
+      <link name="${tf_prefix}suction_cup">
+        <inertial>
+          <origin xyz="0.047500844943701104 0.027424316463654064 -9.637760878256074e-08" rpy="0 0 0"/>
+          <mass value="0.11348172115824295"/>
+          <inertia ixx="2.6e-05" iyy="5.2e-05" izz="6.5e-05" ixy="-2.3e-05" iyz="0.0" ixz="-0.0"/>
+        </inertial>
+        <visual>
+          <origin xyz="-1.19139 -0.578159 -0.71775" rpy="0 0 0"/>
+          <geometry>
+            <mesh filename="file:////home/cem/colcon_ws/src/Universal_Robots_ROS2_Description/meshes/ur10e/secondrobotcollision/suction_cup.stl" scale="0.001 0.001 0.001"/>
+          </geometry>
+          <material name="silver"/>
+        </visual>
+        <collision>
+          <origin xyz="-1.19139 -0.578159 -0.71775" rpy="0 0 0"/>
+          <geometry>
+            <mesh filename="file:////home/cem/colcon_ws/src/Universal_Robots_ROS2_Description/meshes/ur10e/secondrobotcollision/suction_cup.stl" scale="0.001 0.001 0.001"/>
+          </geometry>
+        </collision>
+      </link>
+      <joint name="${tf_prefix}vacuum_gripper_joint" type="fixed">
+        <origin xyz="0.04267 0.056052 -0.0195" rpy="0 0 0"/>
+        <parent link="${tf_prefix}tool0"/>
+        <child link="${tf_prefix}vacuum_gripper"/>
+      </joint>
+      <joint name="${tf_prefix}suction_cup_joint" type="fixed">
+        <origin xyz="0.070588 0.044218 0.0195" rpy="0 0 0"/>
+        <parent link="${tf_prefix}vacuum_gripper"/>
+        <child link="${tf_prefix}suction_cup"/>
+      </joint>
+    </xacro:if>
   </xacro:macro>
 </robot>

File: Universal_Robots_ROS2_Description/urdf/ur_macro.xacro (robot description, xacro)
@@ -85,5 +85,6 @@
     non_blocking_read:=true
     keep_alive_count:=2
-    use_gripper:=false"
+    use_gripper:=false
+    use_vacuum_gripper:=false"
     >
     <!-- Load configuration data from the provided .yaml files -->
@@ -129,4 +130,5 @@
         keep_alive_count="${keep_alive_count}"
         use_gripper="${use_gripper}"
+        use_vacuum_gripper="${use_vacuum_gripper}"
         />
     </xacro:if>
@@ -603,4 +605,57 @@
         use_fake_hardware="$(arg use_fake_hardware)" />
     </xacro:if>
+    <xacro:arg name="use_vacuum_gripper" default="$(optenv ENV_USE_VACUUM_GRIPPER false)"/>
+    <xacro:if value="$(arg use_vacuum_gripper)">
+      <link name="${tf_prefix}vacuum_gripper">
+        <inertial>
+          <origin xyz="0.03840935181996907 0.02553282574514726 0.01947430811837292" rpy="0 0 0"/>
+          <mass value="5.206908838469105"/>
+          <inertia ixx="0.007119" iyy="0.00672" izz="0.006537" ixy="0.000313" iyz="1e-06" ixz="-1e-06"/>
+        </inertial>
+        <visual>
+          <origin xyz="-1.120802 -0.533941 -0.69825" rpy="0 0 0"/>
+          <geometry>
+            <mesh filename="file:////home/cem/colcon_ws/src/Universal_Robots_ROS2_Description/meshes/ur10e/collision/vacuum_gripper.stl" scale="0.001 0.001 0.001"/>
+          </geometry>
+          <material name="silver"/>
+        </visual>
+        <collision>
+          <origin xyz="-1.120802 -0.533941 -0.69825" rpy="0 0 0"/>
+          <geometry>
+            <mesh filename="file:////home/cem/colcon_ws/src/Universal_Robots_ROS2_Description/meshes/ur10e/collision/vacuum_gripper.stl" scale="0.001 0.001 0.001"/>
+          </geometry>
+        </collision>
+      </link>
+      <link name="${tf_prefix}suction_cup">
+        <inertial>
+          <origin xyz="0.047500844943701104 0.027424316463654064 -9.637760878256074e-08" rpy="0 0 0"/>
+          <mass value="0.11348172115824295"/>
+          <inertia ixx="2.6e-05" iyy="5.2e-05" izz="6.5e-05" ixy="-2.3e-05" iyz="0.0" ixz="-0.0"/>
+        </inertial>
+        <visual>
+          <origin xyz="-1.19139 -0.578159 -0.71775" rpy="0 0 0"/>
+          <geometry>
+            <mesh filename="file:////home/cem/colcon_ws/src/Universal_Robots_ROS2_Description/meshes/ur10e/collision/suction_cup.stl" scale="0.001 0.001 0.001"/>
+          </geometry>
+          <material name="silver"/>
+        </visual>
+        <collision>
+          <origin xyz="-1.19139 -0.578159 -0.71775" rpy="0 0 0"/>
+          <geometry>
+            <mesh filename="file:////home/cem/colcon_ws/src/Universal_Robots_ROS2_Description/meshes/ur10e/collision/suction_cup.stl" scale="0.001 0.001 0.001"/>
+          </geometry>
+        </collision>
+      </link>
+      <joint name="${tf_prefix}vacuum_gripper_joint" type="fixed">
+        <origin xyz="0.04267 0.056052 -0.0195" rpy="0 0 0"/>
+        <parent link="${tf_prefix}tool0"/>
+        <child link="${tf_prefix}vacuum_gripper"/>
+      </joint>
+      <joint name="${tf_prefix}suction_cup_joint" type="fixed">
+        <origin xyz="0.070588 0.044218 0.0195" rpy="0 0 0"/>
+        <parent link="${tf_prefix}vacuum_gripper"/>
+        <child link="${tf_prefix}suction_cup"/>
+      </joint>
+    </xacro:if>
   </xacro:macro>
 </robot>

File: mobile_manipulator_description/urdf/ota/ota_plugin.xacro (robot description, xacro)
@@ -1,18 +1,18 @@
 <?xml version="1.0"?>
 <robot xmlns:xacro="http://ros.org/wiki/xacro">
-  <!-- ✅ Joint State Publisher (Ignition: gz-sim-joint-state-publisher-system) -->
+  <!-- ✅ Joint State Publisher (Gazebo Harmonic: gz-sim-joint-state-publisher-system) -->
   <xacro:macro name="ota_joints_state_publisher">
     <gazebo>
-      <plugin filename="libignition-gazebo6-joint-state-publisher-system.so"
-              name="ignition::gazebo::systems::JointStatePublisher">
+      <plugin filename="gz-sim-joint-state-publisher-system"
+              name="gz::sim::systems::JointStatePublisher">
         <update_rate>50</update_rate>
       </plugin>
     </gazebo>
   </xacro:macro>
-  <!-- ✅ Differential Drive Plugin (Ignition: gz-sim-diff-drive-system) -->
+  <!-- ✅ Differential Drive Plugin (Gazebo Harmonic: gz-sim-diff-drive-system) -->
   <xacro:macro name="ota_diff_drive" params="base_link">
     <gazebo>
-      <plugin name="ignition::gazebo::systems::DiffDrive"
-              filename="libignition-gazebo6-diff-drive-system.so">
+      <plugin name="gz::sim::systems::DiffDrive"
+              filename="gz-sim-diff-drive-system">
         <!-- Tekerlek eklemleri (ota_wheel.xacro'daki joint isimleri) -->
         <left_joint>wheel_left_base</left_joint>
