Commit message: Kawasaki-AGV is acting like 7 axis robot

File: Universal_Robots_ROS2_Description/urdf/simrobot_ur_macro.xacro (robot description, xacro)
@@ -609,10 +609,10 @@
       <link name="${tf_prefix}IMX_Camera">
         <inertial>
-          <origin xyz="5.410014880524727e-07 0.008501727362029532 -0.018614321006647505" rpy="0 0 0"/>
-          <mass value="0.044117104706977495"/>
-          <inertia ixx="6e-06" iyy="5e-06" izz="5e-06" ixy="0.0" iyz="0.0" ixz="-0.0"/>
+          <origin xyz="-3.465374807465338e-05 0.0003801084631929186 0.006566275485619721" rpy="0 0 0"/>
+          <mass value="0.04632955033200952"/>
+          <inertia ixx="5e-06" iyy="5e-06" izz="6e-06" ixy="-0.0" iyz="0.0" ixz="-0.0"/>
         </inertial>
         <visual>
-          <origin xyz="-1.078132 -0.499789 -0.70475" rpy="0 0 0"/>
+          <origin xyz="-0.965545 -0.534467 -0.764722" rpy="0 0 0"/>
           <geometry>
             <mesh filename="file:////home/cem/colcon_ws/src/Universal_Robots_ROS2_Description/meshes/ur10e/secondrobotcollision/IMX_Camera.stl" scale="0.001 0.001 0.001"/>
@@ -621,5 +621,5 @@
         </visual>
         <collision>
-          <origin xyz="-1.078132 -0.499789 -0.70475" rpy="0 0 0"/>
+          <origin xyz="-0.965545 -0.534467 -0.764722" rpy="0 0 0"/>
           <geometry>
             <mesh filename="file:////home/cem/colcon_ws/src/Universal_Robots_ROS2_Description/meshes/ur10e/secondrobotcollision/IMX_Camera.stl" scale="0.001 0.001 0.001"/>
@@ -628,10 +628,19 @@
       </link>
       <joint name="${tf_prefix}IMX_Camera_joint" type="fixed">
-        <origin xyz="0.0 -0.038 -0.003" rpy="0 0 0"/>
-        <parent link="${tf_prefix}cable_channel_flange"/>
+        <origin xyz="-0.058785 -0.012133 0.033972" rpy="0 0 0"/>
+        <parent link="${tf_prefix}sick_camera"/>
         <child link="${tf_prefix}IMX_Camera"/>
       </joint>
-      <gazebo reference="${tf_prefix}IMX_Camera">
+      <link name="${tf_prefix}IMX_Camera_frame_link"/>
+      <joint name="${tf_prefix}IMX_Camera_frame_joint" type="fixed">
+        <!-- Datasheet: toplam derinlik 24.68mm, optik merkez lensin önünde -->
+        <origin xyz="0.0 0.025 0.0" rpy="0 0 0" />
+        <parent link="${tf_prefix}IMX_Camera" />
+        <child link="${tf_prefix}IMX_Camera_frame_link"/>
+      </joint>
+      <gazebo reference="${tf_prefix}IMX_Camera_frame_link">
         <sensor name="${tf_prefix}imx179_camera" type="camera">
+          <!-- +Z yönüne bak (roll=-π/2) -->
+          <pose>0 0 0 0 -1.5708 0</pose>
           <always_on>true</always_on>
           <update_rate>30.0</update_rate>
@@ -641,6 +650,6 @@
             <horizontal_fov>2.5307</horizontal_fov>
             <image>
-              <width>3288</width>
-              <height>2512</height>
+              <width>1920</width>
+              <height>1080</height>
               <format>R8G8B8</format>
             </image>
@@ -737,5 +746,5 @@
       <!-- RGBD camera (depth_optical_frame linkine bağlı) -->
       <gazebo reference="${tf_prefix}depth_optical_frame">
-        <sensor name="${tf_prefix}rgbd_camera" type="rgbd_camera">
+        <sensor name="${tf_prefix}depth_optical_frame" type="rgbd_camera">
           <always_on>true</always_on>
           <update_rate>30.0</update_rate>

File: Universal_Robots_ROS2_Tutorials/my_robot_cell/my_robot_cell_control/urdf/whole_cell_real.urdf.xacro (robot description, xacro)
@@ -50,5 +50,5 @@
   <!-- AGV pozisyonu (world frame'e göre) -->
   <xacro:arg name="agv_x" default="-2.301949"/>
-  <xacro:arg name="agv_y" default="0.530401"/>
+  <xacro:arg name="agv_y" default="0.135135131"/>
   <xacro:arg name="agv_z" default="0.17"/>
   <xacro:arg name="agv_yaw" default="1.570796"/>
@@ -60,10 +60,10 @@
   <!-- ==================== 1. AGV + KAWASAKI RS005L (SADECE GÖRSEL/COLLISION) ==================== -->
   <!-- AGV'yi world frame'e sabit bağla -->
-  <joint name="world_to_agv" type="fixed">
+  <!-- <joint name="world_to_agv" type="fixed">
     <parent link="world"/>
     <child link="ota_base_link"/>
     <origin xyz="$(arg agv_x) $(arg agv_y) $(arg agv_z)"
             rpy="0 0 $(arg agv_yaw)"/>
-  </joint>
+  </joint> -->
   <!-- AGV gövdesi (sadece görsel/collision) -->
   <xacro:ota_base link_name="ota_base_link"/>

File: Universal_Robots_ROS2_Tutorials/my_robot_cell/my_robot_cell_control/urdf/whole_cell_sim.urdf.xacro (robot description, xacro)
@@ -62,5 +62,5 @@
   <!-- AGV spawn pozisyonu (world frame'e göre) -->
   <xacro:arg name="agv_x" default="-2.301949"/>
-  <xacro:arg name="agv_y" default="0.530401"/>
+  <xacro:arg name="agv_y" default="0.135135131"/>
   <xacro:arg name="agv_z" default="0.17"/>
   <xacro:arg name="agv_yaw" default="1.570796"/>
@@ -69,10 +69,10 @@
   <!-- ==================== 1. AGV + KAWASAKI RS005L ==================== -->
   <!-- AGV'yi world frame'e sabit bağla (başlangıç pozisyonu) -->
-  <joint name="world_to_agv" type="fixed">
+  <!-- <joint name="world_to_agv" type="fixed">
     <parent link="world"/>
     <child link="ota_base_link"/>
     <origin xyz="$(arg agv_x) $(arg agv_y) $(arg agv_z)"
             rpy="0 0 $(arg agv_yaw)"/>
-  </joint>
+  </joint> -->
   <!-- AGV gövdesi -->
   <xacro:ota_base link_name="ota_base_link"/>

File: Universal_Robots_ROS2_Tutorials/my_robot_cell/my_robot_cell_description/urdf/simrobot_my_robot_cell_macro.xacro (robot description, xacro)
@@ -38,8 +38,8 @@
     </link>
     <!-- Chassis assembly - tüm PART1-PART44 parçalarını içerir -->
-    <!-- <xacro:chassis_assembly tf_prefix="${tf_prefix}" parent="${parent}">
-      <origin xyz="0 0 0" rpy="0 0 0"/>
-    </xacro:chassis_assembly> -->
-    <link name="${tf_prefix}chassis">
+    <xacro:chassis_assembly tf_prefix="${tf_prefix}" parent="${parent}">
+      <origin xyz="0 0 0" rpy="0 0 0"/>
+    </xacro:chassis_assembly>
+    <!-- <link name="${tf_prefix}chassis">
       <inertial>
         <origin xyz="-1.124731 1.232845 1.108302" rpy="0 0 0"/>
@@ -64,5 +64,5 @@
         </geometry>
       </collision>
-    </link>
+    </link> -->
     <link name="${tf_prefix}robot_mount">
       <inertial>
@@ -131,9 +131,9 @@
       <child link="${tf_prefix}table" />
     </joint>
-    <joint name="${tf_prefix}base_to_chassis" type="fixed">
+    <!-- <joint name="${tf_prefix}base_to_chassis" type="fixed">
       <parent link="${parent}"/>
       <child link="${tf_prefix}chassis"/>
       <origin xyz="0 0 0" rpy="0 0 0"/>
-    </joint>
+    </joint> -->
     <!-- Linear axis joint - bu joint'in tam tanımı burada olmalı -->
     <joint name="${tf_prefix}base_to_robot_mount" type="prismatic">

File: mobile_manipulator_description/urdf/ota/ota.ros2_control.xacro (robot description, xacro)
@@ -32,4 +32,16 @@
           <state_interface name="velocity"/>
         </joint>
+        <joint name="world_to_agv">
+          <command_interface name="position"/>
+          <command_interface name="velocity">
+            <param name="min">-1.25</param>
+            <param name="max">1.25</param>
+          </command_interface>
+          <state_interface name="position">
+              <param name="initial_value">1.0</param>
+          </state_interface>
+          <state_interface name="velocity"/>
+          <state_interface name="effort"/>
+        </joint>
       </ros2_control>
     </xacro:if>

File: mobile_manipulator_description/urdf/ota/ota_base.xacro (robot description, xacro)
@@ -2,4 +2,24 @@
 <robot xmlns:xacro="http://ros.org/wiki/xacro">
   <xacro:macro name="ota_base" params="link_name">
+    <!-- <link name="world"/> -->
+    <link name="ifarlab_ray_link">
+      <inertial>
+        <mass value="1.0"/>
+        <inertia ixx="0.001" ixy="0" ixz="0" iyy="0.001" iyz="0" izz="0.001"/>
+      </inertial>
+      <visual>
+        <geometry>
+          <mesh filename="file://$(find mobile_manipulator_description)/meshes/environment/ifarlab_ray.stl" scale="0.001 0.001 0.001"/>
+        </geometry>
+        <material name="ifarlab_ray_material">
+          <color rgba="0.75 0.75 0.75 1"/>
+        </material>
+      </visual>
+      <collision>
+        <geometry>
+          <mesh filename="file://$(find mobile_manipulator_description)/meshes/environment/ifarlab_ray.stl" scale="0.001 0.001 0.001"/>
+        </geometry>
+      </collision>
+    </link>
     <link name='${link_name}'>
       <origin xyz="0 0 0" rpy=" 0 0 0"/>
@@ -65,4 +85,22 @@
       </visual>
     </gazebo> -->
+    <!-- ifarlab.sdf: ifarlab_ray model pose = "0 0 0 0 0 0" → world origin -->
+    <joint name="ifarlab_ray_joint" type="fixed">
+      <parent link="world"/>
+      <child link="ifarlab_ray_link"/>
+      <origin xyz="0 0 0" rpy="0 0 0"/>
+    </joint>
+    <!-- AGV başlangıç konumu: ifarlab.sdf spawn pozisyonundan okundu
+         x=-2.301949  y=0.135135131  z=0.17  yaw=1.570796 (90°)
+         axis 1 0 0 = joint frame local X = yaw 90° nedeniyle world +Y yönü
+         Bu eksende AGV ileri/geri hareket eder (ray üzerinde kayar) -->
+    <joint name="world_to_agv" type="prismatic">
+      <parent link="ifarlab_ray_link"/>
+      <child link="${link_name}"/>
+      <origin xyz="-2.301959 0.135135131 0.165" rpy="0 0 1.570796"/>
+      <axis xyz="1.0 0.0 0.0"/>
+      <limit effort="1000" lower="0.0" upper="2.0" velocity="1.25"/>
+      <dynamics damping="100.0" friction="50.0"/>
+    </joint>
     <joint name="base2manipulatorbase" type="fixed">
       <parent link="${link_name}"/>

Commit message: UseCaseImplementations

File: Universal_Robots_ROS2_Description/urdf/simrobot_ur_macro.xacro (robot description, xacro)
@@ -746,6 +746,6 @@
       <gazebo reference="${tf_prefix}depth_optical_frame">
         <sensor name="${tf_prefix}depth_optical_frame" type="rgbd_camera">
-          <always_on>true</always_on>
-          <update_rate>30.0</update_rate>
+          <always_on>false</always_on>
+          <update_rate>5.0</update_rate>
           <visualize>false</visualize>
           <camera name="${tf_prefix}rgbd">

File: Universal_Robots_ROS2_Tutorials/my_robot_cell/my_robot_cell_description/urdf/my_robot_cell_macro.xacro (robot description, xacro)
@@ -234,10 +234,12 @@
         <material name="silver"/>
       </visual>
-      <collision>
+      <!-- Collision geometry devre dışı: Screwdriver Planning Scene üzerinden
+           attach/detach ile yönetilecek. Gripper kapandığında collision olmasın diye kaldırıldı. -->
+      <!-- <collision>
         <origin rpy="0 0 0" xyz="0 0 0"/>
         <geometry>
           <mesh filename="file:////home/cem/colcon_ws/src/Universal_Robots_ROS2_Description/meshes/ur10e/collision/screwdriver.stl" scale="0.001 0.001 0.001"/>
         </geometry>
-      </collision>
+      </collision> -->
     </link>
     <link name="${tf_prefix}screw_feeder">
