Commit message: Inspection Scenario

File: Universal_Robots_ROS2_Description/urdf/simrobot_ur_macro.xacro (robot description, xacro)
@@ -738,10 +738,10 @@
     <xacro:if value="${sim_ignition}">
       <!-- Sensors system: SADECE 1 KERE -->
-      <gazebo>
-        <plugin filename="ignition-gazebo-sensors-system"
-                name="ignition::gazebo::systems::Sensors">
+     <!-- <gazebo>
+        <plugin filename="gz-sim-sensors-system"
+                name="gz::sim::systems::Sensors">
           <render_engine>ogre2</render_engine>
         </plugin>
-      </gazebo>
+      </gazebo> -->
       <!-- RGBD camera (depth_optical_frame linkine bağlı) -->
       <gazebo reference="${tf_prefix}depth_optical_frame">
@@ -766,4 +766,17 @@
               <far>16.0</far>
             </clip>
+            <!-- Depth noise to approximate the real SICK Visionary-T Mini
+                 (V3S145-1AAAAAA) time-of-flight accuracy. Datasheet
+                 repeatability is ~0.8 mm at 1 m working distance (and ~5 mm at
+                 7 m). SDF applies a *constant* Gaussian sigma, so we use the
+                 near-range figure (0.8 mm = 0.0008 m) matching this task's
+                 0.2-1.0 m inspection distances; real noise grows with range.
+                 Without this the simulated point cloud is perfectly noiseless
+                 and does NOT reflect the physical sensor. -->
+            <noise>
+              <type>gaussian</type>
+              <mean>0.0</mean>
+              <stddev>0.0008</stddev>
+            </noise>
           </camera>
         </sensor>

File: Universal_Robots_ROS2_Tutorials/my_robot_cell/my_robot_cell_description/urdf/chassis_macro.xacro (robot description, xacro)
@@ -14,7 +14,11 @@
         <origin xyz="-1.124731 1.232845 1.108302" rpy="0 0 0"/>
         <mass value="120.90442642947052"/>
-        <inertia ixx="129.47263" ixy="-0.023527" ixz="-0.011644"
-                iyy="73.136591" iyz="-1.726202"
-                izz="85.878511"/>
+        <inertia
+            ixx="1.363e6"
+            ixy="-903.3"
+            ixz="1.847e4"
+            iyy="8.130e5"
+            iyz="-385.3"
+            izz="1.039e6"/>
       </inertial>
     </link>
@@ -31,5 +35,5 @@
           <origin xyz="0 0 0" rpy="0 0 0"/>
           <geometry>
-            <mesh filename="file:////home/cem/colcon_ws/src/Universal_Robots_ROS2_Description/meshes/ur10e/collision/chassis/PART${part_num}.stl" scale="0.001 0.001 0.001"/>
+            <mesh filename="file:////home/cem/colcon_ws/src/Universal_Robots_ROS2_Description/meshes/ur10e/collision/chassis_last/PART${part_num}.stl" scale="0.001 0.001 0.001"/>
           </geometry>
           <material name="${color_material}"/>
@@ -38,5 +42,5 @@
           <origin xyz="0 0 0" rpy="0 0 0"/>
           <geometry>
-            <mesh filename="file:////home/cem/colcon_ws/src/Universal_Robots_ROS2_Description/meshes/ur10e/collision/chassis/PART${part_num}.stl" scale="0.001 0.001 0.001"/>
+            <mesh filename="file:////home/cem/colcon_ws/src/Universal_Robots_ROS2_Description/meshes/ur10e/collision/chassis_last/PART${part_num}.stl" scale="0.001 0.001 0.001"/>
           </geometry>
         </collision>
@@ -72,5 +76,5 @@
     <xacro:chassis_part part_num="15"/>
     <xacro:chassis_part part_num="16"/>
-    <xacro:chassis_part part_num="17" color_material="chassis_red"/>
+    <xacro:chassis_part part_num="17"/>
     <xacro:chassis_part part_num="18"/>
     <xacro:chassis_part part_num="19"/>
@@ -83,5 +87,5 @@
     <xacro:chassis_part part_num="26"/>
     <xacro:chassis_part part_num="27"/>
-    <xacro:chassis_part part_num="28"/>
+    <xacro:chassis_part part_num="28" color_material="chassis_red"/>
     <xacro:chassis_part part_num="29"/>
     <xacro:chassis_part part_num="30"/>
@@ -100,8 +104,21 @@
     <xacro:chassis_part part_num="43"/>
     <xacro:chassis_part part_num="44"/>
+    <xacro:chassis_part part_num="45"/>
+    <xacro:chassis_part part_num="46"/>
+    <xacro:chassis_part part_num="47"/>
+    <xacro:chassis_part part_num="48"/>
+    <xacro:chassis_part part_num="49"/>
+    <xacro:chassis_part part_num="50"/>
+    <xacro:chassis_part part_num="51"/>
+    <xacro:chassis_part part_num="52"/>
+    <xacro:chassis_part part_num="53"/>
+    <xacro:chassis_part part_num="54"/>
+    <xacro:chassis_part part_num="55"/>
+    <xacro:chassis_part part_num="56"/>
+    <xacro:chassis_part part_num="57"/>
     <!-- Gazebo için renk tanımlamaları -->
-    <gazebo reference="${tf_prefix}chassis_part17">
+    <!-- <gazebo reference="${tf_prefix}chassis_part17">
       <material>Gazebo/Red</material>
-    </gazebo>
+    </gazebo> -->
     <!-- <gazebo reference="${tf_prefix}chassis_part23">
       <material>Gazebo/Red</material>

File: Universal_Robots_ROS2_Tutorials/my_robot_cell/my_robot_cell_description/urdf/my_robot_cell_macro.xacro (robot description, xacro)
@@ -48,8 +48,8 @@
     </link>
     <!-- Chassis assembly - tüm PART1-PART44 parçalarını içerir -->
-    <!-- <xacro:chassis_assembly tf_prefix="${tf_prefix}" parent="${parent}">
-      <origin xyz="0 0 0" rpy="0 0 0"/>
-    </xacro:chassis_assembly> -->
-    <link name="${tf_prefix}chassis">
+    <xacro:chassis_assembly tf_prefix="${tf_prefix}" parent="${parent}">
+      <origin xyz="0 0 0" rpy="0 0 0"/>
+    </xacro:chassis_assembly>
+    <!-- <link name="${tf_prefix}chassis">
       <inertial>
         <origin xyz="-1.124731 1.232845 1.108302" rpy="0 0 0"/>
@@ -80,5 +80,5 @@
         </geometry>
       </collision>
-    </link>
+    </link> -->
     <!-- Platform - Bodies(1): mass=205.0 kg, inertia CAD'dan alındı -->
     <!-- <link name="${tf_prefix}platform">
@@ -293,9 +293,9 @@
       <dynamics damping="100.0" friction="50.0"/>
     </joint>
-    <joint name="${tf_prefix}base_to_chassis" type="fixed">
+    <!-- <joint name="${tf_prefix}base_to_chassis" type="fixed">
       <parent link="${parent}"/>
       <child link="${tf_prefix}chassis"/>
       <origin xyz="0 0 0" rpy="0 0 0"/>
-    </joint>
+    </joint> -->
     <!-- <joint name="${tf_prefix}base_to_platform" type="fixed">
       <parent link="${parent}"/>

File: Universal_Robots_ROS2_Tutorials/my_robot_cell/my_robot_cell_description/urdf/simrobot_my_robot_cell_macro.xacro (robot description, xacro)
@@ -38,10 +38,8 @@
       </collision>
     </link>
-    <!-- Chassis assembly - devre dışı bırakıldı, platform/door/door1 ile değiştirildi
     <xacro:chassis_assembly tf_prefix="${tf_prefix}" parent="${parent}">
       <origin xyz="0 0 0" rpy="0 0 0"/>
     </xacro:chassis_assembly>
-    -->
-    <link name="${tf_prefix}chassis">
+    <!-- <link name="${tf_prefix}chassis">
       <inertial>
         <origin xyz="-1.124731 1.232845 1.108302" rpy="0 0 0"/>
@@ -72,5 +70,5 @@
         </geometry>
       </collision>
-    </link>
+    </link> -->
     <!-- Platform - Bodies(1): mass=205.0 kg, inertia CAD'dan alındı -->
     <!-- <link name="${tf_prefix}platform">
@@ -248,9 +246,9 @@
       <child link="${tf_prefix}table" />
     </joint>
-    <joint name="${tf_prefix}base_to_chassis" type="fixed">
+    <!-- <joint name="${tf_prefix}base_to_chassis" type="fixed">
       <parent link="${parent}"/>
       <child link="${tf_prefix}chassis"/>
       <origin xyz="0 0 0" rpy="0 0 0"/>
-    </joint>
+    </joint> -->
     <!-- <joint name="${tf_prefix}base_to_platform" type="fixed">
       <parent link="${parent}"/>

File: mobile_manipulator_description/urdf/khi_rs/rs005l_macro.xacro (robot description, xacro)
@@ -196,5 +196,5 @@
           <mesh filename="package://mobile_manipulator_description/meshes/khi_rs/RS005L_J6.STL"/>
         </geometry>
-        <material name="Black"/>
+        <material name="White"/>
         <origin xyz="0 0 0" rpy="0 0 0"/>
       </visual>
@@ -203,8 +203,25 @@
           <mesh filename="package://mobile_manipulator_description/meshes/khi_rs/RS005L_J6.STL"/>
         </geometry>
-        <material name="Black"/>
+        <material name="White"/>
         <origin xyz="0 0 0" rpy="0 0 0"/>
       </collision>
       <xacro:default_inertial mass="${j6_mass}"/>
+    </link>
+    <link name="${tf_prefix}link7">
+      <visual>
+        <geometry>
+          <mesh filename="package://mobile_manipulator_description/meshes/khi_rs/Montaj.stl" scale="0.001 0.001 0.001"/>
+        </geometry>
+        <material name="White"/>
+        <origin xyz="-0.035 -0.04 0.2175" rpy="1.570796 3.1415 0"/>
+      </visual>
+      <collision>
+        <geometry>
+          <mesh filename="package://mobile_manipulator_description/meshes/khi_rs/Montaj.stl" scale="0.001 0.001 0.001"/>
+        </geometry>
+        <material name="White"/>
+        <origin xyz="-0.035 -0.04 0.2175" rpy="1.570796 3.1415 0"/>
+      </collision>
+      <xacro:default_inertial mass="0.1"/>
     </link>
     <!-- === Link 1 === -->
@@ -262,5 +279,69 @@
       <dynamics damping="0.0" friction="0.0"/>
     </joint>
-    <!-- ÇEVRESEL BİLEŞENLER -->
+    <joint name="${tf_prefix}joint7" type="fixed">
+      <axis xyz="0 0 1" rpy="0 0 0" />
+      <origin xyz="0 0 0" rpy="0 0 -1.96" />
+      <parent link="${tf_prefix}link6"/>
+      <child link="${tf_prefix}link7"/>
+    </joint>
+    <link name="${tf_prefix}camera_link">
+      <inertial>
+        <mass value="0.01"/>
+        <origin xyz="0 0 0" rpy="0 0 0"/>
+        <inertia ixx="0.0001" ixy="0" ixz="0" iyy="0.0001" iyz="0" izz="0.0001"/>
+      </inertial>
+    </link>
+    <joint name="${tf_prefix}camera_joint" type="fixed">
+       <origin xyz="0.0145 0.0125 0.185" rpy="0 -1.570796 1.570796"/>
+       <parent link="${tf_prefix}link7"/>
+       <child link="${tf_prefix}camera_link"/>
+    </joint>
+    <joint name="${tf_prefix}camera_rgb_joint" type="fixed">
+       <origin xyz="0 0 0" rpy="0 0 0"/>
+       <parent link="${tf_prefix}camera_link"/>
+       <child link="${tf_prefix}camera_rgb_frame"/>
+    </joint>
+    <link name="${tf_prefix}camera_rgb_frame"/>
+    <joint name="${tf_prefix}camera_rgb_optic_joint" type="fixed">
+       <origin xyz="0 0 0" rpy="0 0 0"/>
+       <parent link="${tf_prefix}camera_rgb_frame"/>
+       <child link="${tf_prefix}camera_rgb_optic_frame"/>
+    </joint>
+    <link name="${tf_prefix}camera_rgb_optic_frame"/>
+    <xacro:if value="${sim_ignition}">
+      <!-- NOT: gz-sim-sensors-system plugin'i world SDF'de (ifarlab.sdf) zaten
+           yükleniyor. Burada tekrar tanımlamak "Scene already exists" hatasına
+           ve ardından WaitForInit() segfault'una yol açar. Sadece sensör
+           tanımı (<gazebo reference=...>) yeterlidir. -->
+      <gazebo reference="${tf_prefix}camera_rgb_optic_frame">
+        <sensor name="${tf_prefix}camera_rgb_optic_frame" type="rgbd_camera">
+          <always_on>false</always_on>
+          <update_rate>5.0</update_rate>
+          <visualize>false</visualize>
+          <camera name="${tf_prefix}rgbd">
+            <horizontal_fov>1.22</horizontal_fov>
+            <image>
+              <width>512</width>
+              <height>424</height>
+              <format>R8G8B8</format>
+            </image>
+            <depth_image>
+              <width>512</width>
+              <height>424</height>
+              <format>R_FLOAT32</format>
+            </depth_image>
+            <clip>
+              <near>0.05</near>
+              <far>16.0</far>
+            </clip>
+            <noise>
+              <type>gaussian</type>
+              <mean>0.0</mean>
+              <stddev>0.0008</stddev>
+            </noise>
+          </camera>
+        </sensor>
+      </gazebo>
+    </xacro:if>
   </xacro:macro>
 </robot>

File: rs005l_description/urdf/rs005l_macro.xacro (robot description, xacro)
@@ -244,4 +244,32 @@
       <dynamics friction="0.1"/>
     </joint>
+    <joint name="${tf_prefix}joint7" type="fixed">
+      <axis xyz="0 0 1" rpy="0 0 0" />
+      <origin xyz="0 0 0" rpy="0 0 -1.96" />
+      <parent link="${tf_prefix}link6"/>
+      <child link="${tf_prefix}link7"/>
+    </joint>
+    <link name="${tf_prefix}link7">
+      <inertial>
+        <origin xyz="5.0628E-17 -4.215E-14 0.074772" rpy="0 0 0"/>
+        <mass value="0.0065669"/>
+        <inertia ixx="743E-09" ixy="0E-09" ixz="0E-09" iyy="743E-09" iyz="0E-09" izz="1448E-09"/>
+      </inertial>
+      <visual>
+        <origin xyz="0 0 0.078" rpy="0 0 0"/>
+        <geometry>
+          <mesh filename="file:////home/cem/colcon_ws/src/rs005l_description/meshes/Montaj.stl" scale="0.001 0.001 0.001"/>
+        </geometry>
+        <material name="">
+          <color rgba="0.79216 0.81961 0.93333 1"/>
+        </material>
+      </visual>
+      <collision>
+        <origin xyz="0 0 0.078" rpy="0 0 0"/>
+        <geometry>
+          <mesh filename="file:////home/cem/colcon_ws/src/rs005l_description/meshes/Montaj.stl" scale="0.001 0.001 0.001"/>
+        </geometry>
+      </collision>
+    </link>
     <transmission name="tran1">
       <plugin>transmission_interface/SimpleTransmission</plugin>
