Commit message: Harmony+Multi-Robot Inspection

File: Universal_Robots_ROS2_Description/urdf/simrobot_ur_macro.xacro (robot description, xacro)
@@ -499,4 +499,36 @@
         </geometry>
       </collision>
+      <!-- SICK camera collision shell (identical to the real ur_macro.xacro).
+           The mesh above under-reports the real housing, so these six boxes
+           wrap it on all sides: front (optics face), back, and four sides,
+           yawed 60 deg about the viewing axis to match the housing. All four
+           neighbour links (flange, tool0, cable_channel, cable_channel_flange)
+           are already disabled against sick_camera in every SRDF, so these add
+           no permanent self-collision. Formerly attached at runtime in
+           ur_inspection_node._setup_planning_scene_extras. -->
+      <collision>
+        <origin xyz="-0.0301 0.0174 0.0537" rpy="0 0 1.047198"/>
+        <geometry><box size="0.087 0.090 0.039"/></geometry>
+      </collision>
+      <collision>
+        <origin xyz="-0.0301 0.0174 -0.0628" rpy="0 0 1.047198"/>
+        <geometry><box size="0.087 0.090 0.039"/></geometry>
+      </collision>
+      <collision>
+        <origin xyz="0.0014 0.071959 -0.00455" rpy="0 0 1.047198"/>
+        <geometry><box size="0.039 0.090 0.0775"/></geometry>
+      </collision>
+      <collision>
+        <origin xyz="-0.0616 -0.037159 -0.00455" rpy="0 0 1.047198"/>
+        <geometry><box size="0.039 0.090 0.0775"/></geometry>
+      </collision>
+      <collision>
+        <origin xyz="-0.085959 0.04965 -0.00455" rpy="0 0 1.047198"/>
+        <geometry><box size="0.087 0.039 0.0775"/></geometry>
+      </collision>
+      <collision>
+        <origin xyz="0.025759 -0.01485 -0.00455" rpy="0 0 1.047198"/>
+        <geometry><box size="0.087 0.039 0.0775"/></geometry>
+      </collision>
     </link>
     <joint name="${tf_prefix}flange-tool0" type="fixed">

File: Universal_Robots_ROS2_Description/urdf/ur_macro.xacro (robot description, xacro)
@@ -500,4 +500,40 @@
         </geometry>
       </collision>
+      <!-- SICK camera collision shell. The mesh above under-reports the real
+           housing (its front face stops ~1.9 cm short of the physical optics
+           cover), so MoveIt used to plan the camera into the UR's own joints
+           and the cable channel. These six boxes wrap the housing on all
+           sides: front (optics face), back, and the four sides. They are
+           yawed 60 deg about the viewing axis to match the housing (same angle
+           as ur_sick_optical_joint's rpy). All four neighbour links
+           (flange, tool0, cable_channel, cable_channel_flange) are already
+           disabled against sick_camera in every SRDF, so these boxes add no
+           permanent self-collision. Front/back = 8.7 x 9.0 x 3.9 cm skirts;
+           sides span the 7.75 cm housing depth. Formerly attached at runtime
+           in ur_inspection_node._setup_planning_scene_extras. -->
+      <collision>
+        <origin xyz="-0.0301 0.0174 0.0537" rpy="0 0 1.047198"/>
+        <geometry><box size="0.087 0.090 0.039"/></geometry>
+      </collision>
+      <collision>
+        <origin xyz="-0.0301 0.0174 -0.0628" rpy="0 0 1.047198"/>
+        <geometry><box size="0.087 0.090 0.039"/></geometry>
+      </collision>
+      <collision>
+        <origin xyz="0.0014 0.071959 -0.00455" rpy="0 0 1.047198"/>
+        <geometry><box size="0.039 0.090 0.0775"/></geometry>
+      </collision>
+      <collision>
+        <origin xyz="-0.0616 -0.037159 -0.00455" rpy="0 0 1.047198"/>
+        <geometry><box size="0.039 0.090 0.0775"/></geometry>
+      </collision>
+      <collision>
+        <origin xyz="-0.085959 0.04965 -0.00455" rpy="0 0 1.047198"/>
+        <geometry><box size="0.087 0.039 0.0775"/></geometry>
+      </collision>
+      <collision>
+        <origin xyz="0.025759 -0.01485 -0.00455" rpy="0 0 1.047198"/>
+        <geometry><box size="0.087 0.039 0.0775"/></geometry>
+      </collision>
     </link>
     <link name="${tf_prefix}cable_channel_flange">

File: Universal_Robots_ROS2_Tutorials/my_robot_cell/my_robot_cell_description/urdf/my_robot_cell_macro.xacro (robot description, xacro)
@@ -48,7 +48,7 @@
     </link>
     <!-- Chassis assembly - tüm PART1-PART44 parçalarını içerir -->
-    <xacro:chassis_assembly tf_prefix="${tf_prefix}" parent="${parent}">
-      <origin xyz="0 0 0" rpy="0 0 0"/>
-    </xacro:chassis_assembly>
+    <!-- <xacro:chassis_assembly tf_prefix="${tf_prefix}" parent="${parent}">
+      <origin xyz="0 0 0" rpy="0 0 0"/>
+    </xacro:chassis_assembly> -->
     <!-- <link name="${tf_prefix}chassis">
       <inertial>
@@ -82,5 +82,5 @@
     </link> -->
     <!-- Platform - Bodies(1): mass=205.0 kg, inertia CAD'dan alındı -->
-    <!-- <link name="${tf_prefix}platform">
+    <link name="${tf_prefix}platform">
       <inertial>
         <origin xyz="-1.101122 1.387607 0.574201" rpy="0 0 0"/>
@@ -93,17 +93,17 @@
         <origin xyz="0 0 0" rpy="0 0 0"/>
         <geometry>
-          <mesh filename="file:////home/cem/colcon_ws/src/Universal_Robots_ROS2_Description/meshes/ur10e/collision/platform.stl" scale="0.001 0.001 0.001"/>
-        </geometry>
-        <material name="silver"/>
-      </visual>
-      <collision>
-        <origin xyz="0 0 0" rpy="0 0 0"/>
-        <geometry>
-          <mesh filename="file:////home/cem/colcon_ws/src/Universal_Robots_ROS2_Description/meshes/ur10e/collision/platform.stl" scale="0.001 0.001 0.001"/>
-        </geometry>
-      </collision>
-    </link> -->
+          <mesh filename="file:////home/cem/colcon_ws/src/Universal_Robots_ROS2_Description/meshes/ur10e/collision/platform.stl" scale="1 1 1"/>
+        </geometry>
+        <material name="silver"/>
+      </visual>
+      <collision>
+        <origin xyz="0 0 0" rpy="0 0 0"/>
+        <geometry>
+          <mesh filename="file:////home/cem/colcon_ws/src/Universal_Robots_ROS2_Description/meshes/ur10e/collision/platform.stl" scale="1 1 1"/>
+        </geometry>
+      </collision>
+    </link>
     <!-- Door - araba kapısı (~18 kg, 1.1m x 0.9m x 0.05m çelik) -->
-    <!-- <link name="${tf_prefix}windowlessdoor">
+    <link name="${tf_prefix}windowlessdoor">
       <inertial>
         <origin xyz="-0.864306 0.816343 0.934094" rpy="0 0 0"/>
@@ -116,17 +116,17 @@
         <origin xyz="0 0 0" rpy="0 0 0"/>
         <geometry>
-          <mesh filename="file:////home/cem/colcon_ws/src/Universal_Robots_ROS2_Description/meshes/ur10e/collision/windowlessdoor.stl" scale="0.001 0.001 0.001"/>
-        </geometry>
-        <material name="silver"/>
-      </visual>
-      <collision>
-        <origin xyz="0 0 0" rpy="0 0 0"/>
-        <geometry>
-          <mesh filename="file:////home/cem/colcon_ws/src/Universal_Robots_ROS2_Description/meshes/ur10e/collision/windowlessdoor.stl" scale="0.001 0.001 0.001"/>
-        </geometry>
-      </collision>
-    </link> -->
+          <mesh filename="file:////home/cem/colcon_ws/src/Universal_Robots_ROS2_Description/meshes/ur10e/collision/windowlessdoor.stl" scale="1 1 1"/>
+        </geometry>
+        <material name="silver"/>
+      </visual>
+      <collision>
+        <origin xyz="0 0 0" rpy="0 0 0"/>
+        <geometry>
+          <mesh filename="file:////home/cem/colcon_ws/src/Universal_Robots_ROS2_Description/meshes/ur10e/collision/windowlessdoor.stl" scale="1 1 1"/>
+        </geometry>
+      </collision>
+    </link>
     <!-- Door1 - araba kapısı (~18 kg, 1.1m x 0.9m x 0.05m çelik) -->
-    <!-- <link name="${tf_prefix}windowdoor">
+    <link name="${tf_prefix}windowdoor">
       <inertial>
         <origin xyz="-0.844038 1.994389 0.74421" rpy="0 0 0"/>
@@ -139,15 +139,15 @@
         <origin xyz="0 0 0" rpy="0 0 0"/>
         <geometry>
-          <mesh filename="file:////home/cem/colcon_ws/src/Universal_Robots_ROS2_Description/meshes/ur10e/collision/windowdoor.stl" scale="0.001 0.001 0.001"/>
-        </geometry>
-        <material name="silver"/>
-      </visual>
-      <collision>
-        <origin xyz="0 0 0" rpy="0 0 0"/>
-        <geometry>
-          <mesh filename="file:////home/cem/colcon_ws/src/Universal_Robots_ROS2_Description/meshes/ur10e/collision/windowdoor.stl" scale="0.001 0.001 0.001"/>
-        </geometry>
-      </collision>
-    </link> -->
+          <mesh filename="file:////home/cem/colcon_ws/src/Universal_Robots_ROS2_Description/meshes/ur10e/collision/windowdoor.stl" scale="1 1 1"/>
+        </geometry>
+        <material name="silver"/>
+      </visual>
+      <collision>
+        <origin xyz="0 0 0" rpy="0 0 0"/>
+        <geometry>
+          <mesh filename="file:////home/cem/colcon_ws/src/Universal_Robots_ROS2_Description/meshes/ur10e/collision/windowdoor.stl" scale="1 1 1"/>
+        </geometry>
+      </collision>
+    </link>
     <link name="${tf_prefix}robot_mount">
       <inertial>
@@ -298,5 +298,5 @@
       <origin xyz="0 0 0" rpy="0 0 0"/>
     </joint> -->
-    <!-- <joint name="${tf_prefix}base_to_platform" type="fixed">
+    <joint name="${tf_prefix}base_to_platform" type="fixed">
       <parent link="${parent}"/>
       <child link="${tf_prefix}platform"/>
@@ -312,5 +312,5 @@
       <child link="${tf_prefix}windowdoor"/>
       <origin xyz="0 0 0" rpy="0 0 0"/>
-    </joint> -->
+    </joint>
     <joint name="${tf_prefix}base_to_alumuniumtable" type="fixed">
       <parent link="${parent}"/>

File: Universal_Robots_ROS2_Tutorials/my_robot_cell/my_robot_cell_description/urdf/simrobot_my_robot_cell_macro.xacro (robot description, xacro)
@@ -38,7 +38,7 @@
       </collision>
     </link>
-    <xacro:chassis_assembly tf_prefix="${tf_prefix}" parent="${parent}">
-      <origin xyz="0 0 0" rpy="0 0 0"/>
-    </xacro:chassis_assembly>
+    <!-- <xacro:chassis_assembly tf_prefix="${tf_prefix}" parent="${parent}">
+      <origin xyz="0 0 0" rpy="0 0 0"/>
+    </xacro:chassis_assembly> -->
     <!-- <link name="${tf_prefix}chassis">
       <inertial>
@@ -72,5 +72,5 @@
     </link> -->
     <!-- Platform - Bodies(1): mass=205.0 kg, inertia CAD'dan alındı -->
-    <!-- <link name="${tf_prefix}platform">
+    <link name="${tf_prefix}platform">
       <inertial>
         <origin xyz="-1.101122 1.387607 0.574201" rpy="0 0 0"/>
@@ -83,17 +83,17 @@
         <origin xyz="0 0 0" rpy="0 0 0"/>
         <geometry>
-          <mesh filename="file:////home/cem/colcon_ws/src/Universal_Robots_ROS2_Description/meshes/ur10e/collision/platform.stl" scale="0.001 0.001 0.001"/>
-        </geometry>
-        <material name="silver"/>
-      </visual>
-      <collision>
-        <origin xyz="0 0 0" rpy="0 0 0"/>
-        <geometry>
-          <mesh filename="file:////home/cem/colcon_ws/src/Universal_Robots_ROS2_Description/meshes/ur10e/collision/platform.stl" scale="0.001 0.001 0.001"/>
-        </geometry>
-      </collision>
-    </link> -->
+          <mesh filename="file:////home/cem/colcon_ws/src/Universal_Robots_ROS2_Description/meshes/ur10e/collision/platform.stl" scale="1 1 1"/>
+        </geometry>
+        <material name="silver"/>
+      </visual>
+      <collision>
+        <origin xyz="0 0 0" rpy="0 0 0"/>
+        <geometry>
+          <mesh filename="file:////home/cem/colcon_ws/src/Universal_Robots_ROS2_Description/meshes/ur10e/collision/platform.stl" scale="1 1 1"/>
+        </geometry>
+      </collision>
+    </link>
     <!-- Door - araba kapısı (~18 kg, 1.1m x 0.9m x 0.05m çelik) -->
-    <!-- <link name="${tf_prefix}windowlessdoor">
+    <link name="${tf_prefix}windowlessdoor">
       <inertial>
         <origin xyz="-0.864306 0.816343 0.934094" rpy="0 0 0"/>
@@ -106,17 +106,17 @@
         <origin xyz="0 0 0" rpy="0 0 0"/>
         <geometry>
-          <mesh filename="file:////home/cem/colcon_ws/src/Universal_Robots_ROS2_Description/meshes/ur10e/collision/windowlessdoor.stl" scale="0.001 0.001 0.001"/>
-        </geometry>
-        <material name="silver"/>
-      </visual>
-      <collision>
-        <origin xyz="0 0 0" rpy="0 0 0"/>
-        <geometry>
-          <mesh filename="file:////home/cem/colcon_ws/src/Universal_Robots_ROS2_Description/meshes/ur10e/collision/windowlessdoor.stl" scale="0.001 0.001 0.001"/>
-        </geometry>
-      </collision>
-    </link> -->
+          <mesh filename="file:////home/cem/colcon_ws/src/Universal_Robots_ROS2_Description/meshes/ur10e/collision/windowlessdoor.stl" scale="1 1 1"/>
+        </geometry>
+        <material name="silver"/>
+      </visual>
+      <collision>
+        <origin xyz="0 0 0" rpy="0 0 0"/>
+        <geometry>
+          <mesh filename="file:////home/cem/colcon_ws/src/Universal_Robots_ROS2_Description/meshes/ur10e/collision/windowlessdoor.stl" scale="1 1 1"/>
+        </geometry>
+      </collision>
+    </link>
     <!-- Door1 - araba kapısı (~18 kg, 1.1m x 0.9m x 0.05m çelik) -->
-    <!-- <link name="${tf_prefix}windowdoor">
+    <link name="${tf_prefix}windowdoor">
       <inertial>
         <origin xyz="-0.844038 1.994389 0.74421" rpy="0 0 0"/>
@@ -129,15 +129,15 @@
         <origin xyz="0 0 0" rpy="0 0 0"/>
         <geometry>
-          <mesh filename="file:////home/cem/colcon_ws/src/Universal_Robots_ROS2_Description/meshes/ur10e/collision/windowdoor.stl" scale="0.001 0.001 0.001"/>
-        </geometry>
-        <material name="silver"/>
-      </visual>
-      <collision>
-        <origin xyz="0 0 0" rpy="0 0 0"/>
-        <geometry>
-          <mesh filename="file:////home/cem/colcon_ws/src/Universal_Robots_ROS2_Description/meshes/ur10e/collision/windowdoor.stl" scale="0.001 0.001 0.001"/>
-        </geometry>
-      </collision>
-    </link> -->
+          <mesh filename="file:////home/cem/colcon_ws/src/Universal_Robots_ROS2_Description/meshes/ur10e/collision/windowdoor.stl" scale="1 1 1"/>
+        </geometry>
+        <material name="silver"/>
+      </visual>
+      <collision>
+        <origin xyz="0 0 0" rpy="0 0 0"/>
+        <geometry>
+          <mesh filename="file:////home/cem/colcon_ws/src/Universal_Robots_ROS2_Description/meshes/ur10e/collision/windowdoor.stl" scale="1 1 1"/>
+        </geometry>
+      </collision>
+    </link>
     <link name="${tf_prefix}robot_mount">
       <inertial>
@@ -251,5 +251,5 @@
       <origin xyz="0 0 0" rpy="0 0 0"/>
     </joint> -->
-    <!-- <joint name="${tf_prefix}base_to_platform" type="fixed">
+    <joint name="${tf_prefix}base_to_platform" type="fixed">
       <parent link="${parent}"/>
       <child link="${tf_prefix}platform"/>
@@ -265,5 +265,5 @@
       <child link="${tf_prefix}windowdoor"/>
       <origin xyz="0 0 0" rpy="0 0 0"/>
-    </joint> -->
+    </joint>
     <!-- Linear axis joint - bu joint'in tam tanımı burada olmalı -->
     <joint name="${tf_prefix}base_to_robot_mount" type="prismatic">
